File: _Projects/P1012202501-ESP32_Stepper_Controller/Hardware/P1012202501-ESP32_Stepper_Controller/P1012202501-ESP32_Stepper_Controller.kicad_sch (KiCad schematic)
At the start: 7 parts, among them IC1 PMAP63203WU-7

Commit message: Adding all updated files from latest stream.
Parts:
- added C10, C9: CC1210226025AAAX7R, COMPONENTS:CAP-1210, symbol COMPONENTS:CC1210226025AAAX7R
- added C6, C7: CC1206106050AAAX7R, COMPONENTS:CAP-1206, symbol COMPONENTS:CC1206106050AAAX7R
- added C8: CC0603104050AAAX7R, COMPONENTS:CAP-0603, symbol COMPONENTS:CC0603104050AAAX7R
- added IC2: PMAP63205WU-7, COMPONENTS:TSOT-26-6, symbol COMPONENTS:PMAP63205WU-7
- added L2: LSRP2512-2R2M, COMPONENTS:IND-1005, symbol COMPONENTS:LSRP2512-2R2M
Connections:
- net +24V: now also C6.1, C7.1, IC2.2 (EN), IC2.3 (VIN)
- net GND: now also C10.2, C6.2, C7.2, C9.2, IC2.4 (GND)
- new net: C8.2, IC2.5 (SW), L2.1
- new net: C8.1, IC2.6 (BST)
- new net +5V: C10.1, C9.1, IC2.1 (FB), L2.2
Other:
- added sheet ESP32 (untitled.kicad_sch)
