File: _Projects/P1012202501-ESP32_Stepper_Controller/Hardware/P1012202501-ESP32_Stepper_Controller/P1012202501-ESP32_Stepper_Controller.kicad_sch (KiCad schematic)
At the start: 6 parts

Commit message: Added new items from stream.
Parts:
- added LGO1: ~, LOGOS:Logo10x40mm, symbol LOGOS:LOGO10x40mm
- added MH1, MH2, MH3, MH4: ~, HARDWARE:M3MountingHole, symbol HARDWARE:M3MountingHole
- FID1, FID6: value ~ -> (none); footprint (none) -> COMPONENTS:FID1.0x1.5mm Round
- FID2: renamed from FID4; value ~ -> (none); footprint (none) -> COMPONENTS:FID1.0x1.5mm Round
- FID3: renamed from FID2; value ~ -> (none); footprint (none) -> COMPONENTS:FID1.0x1.5mm Round
- FID4: renamed from FID5; value ~ -> (none); footprint (none) -> COMPONENTS:FID1.0x1.5mm Round
- FID5: renamed from FID3; value ~ -> (none); footprint (none) -> COMPONENTS:FID1.0x1.5mm Round
Connections:
- no-connect marks 0 -> 4
Other:
- note added: "MOUNTING HARDWARE"

Commit message: Added new content and changes from stream.
Parts:
- FID1, FID2, FID3, FID4, FID5, FID6: value (none) -> ~
Changed lines of the file:
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@@
 			)
 		)
-		(property "Value" ""
+		(property "Value" "~"
 			(at 246.38 151.13 0)
 			(effects
@@
 			)
 		)
-		(property "Value" ""
+		(property "Value" "~"
 			(at 259.08 151.13 0)
 			(effects
@@
 			)
 		)
-		(property "Value" ""
+		(property "Value" "~"
 			(at 270.51 158.75 0)
 			(effects
@@
 			)
 		)
-		(property "Value" ""
+		(property "Value" "~"
 			(at 246.38 158.75 0)
 			(effects
@@
 			)
 		)
-		(property "Value" ""
+		(property "Value" "~"
 			(at 259.08 158.75 0)
 			(effects
@@
 			)
 		)
-		(property "Value" ""
+		(property "Value" "~"
 			(at 270.51 151.13 0)
 			(effects

Commit message: Added new content from stream.
Other:
- note added: "2"
Changed lines of the file:
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@@
+		)
+	)
+	(text "2"
+		(exclude_from_sim no)
+		(at 269.24 193.548 0)
+		(effects
+			(font
+				(size 1.27 1.27)
+			)
 		)
 	)

Commit message: Added new items from recent stream.
Other:
- added sheet Changelog (P1012202501-Changelog.kicad_sch)
- added sheet Test Point Index (P1012202501-Test Point Index.kicad_sch)
Changed lines of the file:
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@@
+	)
+	(sheet
+		(at 97.79 45.72)
+		(size 12.7 13.97)
+		(exclude_from_sim no)
+		(in_bom yes)
+		(on_board yes)
+		(dnp no)
+		(fields_autoplaced yes)
+		(stroke
+			(width 0.1524)
+			(type solid)
+		)
+		(fill
+			(color 0 0 0 0.0000)
+		)
+		(property "Sheetname" "Changelog"
+			(at 97.79 45.0084 0)
+			(effects
+				(font
+					(size 1.27 1.27)
+				)
+				(justify left bottom)
+			)
+		)
+		(property "Sheetfile" "P1012202501-Changelog.kicad_sch"
+			(at 97.79 60.2746 0)
+			(effects
+				(font
+					(size 1.27 1.27)
+				)
+				(justify left top)
+			)
+		)
+		(instances
+			(project "P1012202501-ESP32_Stepper_Controller"
+				(path "/27f0531a-0a2b-4c68-af50-4332bf165b5a"
+					(page "10")
+				)
+			)
+		)
 	)
 	(sheet
@@
 				)
 			)
+		)
+	)
+	(sheet
+		(at 97.79 25.4)
+		(size 12.7 13.97)
+		(exclude_from_sim no)
+		(in_bom yes)
+		(on_board yes)
+		(dnp no)
+		(fields_autoplaced yes)
+		(stroke
+			(width 0.1524)
+			(type solid)
+		)
+		(fill
+			(color 0 0 0 0.0000)
+		)
+		(property "Sheetname" "Test Point Index"
+			(at 97.79 24.6884 0)
+			(effects
+				(font
+					(size 1.27 1.27)
+				)
+				(justify left bottom)
+			)
+		)
+		(property "Sheetfile" "P1012202501-Test Point Index.kicad_sch"
+			(at 97.79 39.9546 0)
+			(effects
+				(font
+					(size 1.27 1.27)
+				)
+				(justify left top)
+			)
+		)
+		(instances
+			(project "P1012202501-ESP32_Stepper_Controller"
+				(path "/27f0531a-0a2b-4c68-af50-4332bf165b5a"
+					(page "9")
+				)
+			)
