File: _Projects/P1012202501-ESP32_Stepper_Controller/Hardware/P1012202501-ESP32_Stepper_Controller/P1012202501-Cover Sheet.kicad_sch (KiCad schematic)
At the start: 0 parts

Commit message: Added content from latest stream.
Other:
- added sheet RS-485 (P1012202501-RS-485.kicad_sch)
Changed lines of the file:
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@@
+		)
+	)
+	(sheet
+		(at 38.1 68.58)
+		(size 13.97 13.97)
+		(exclude_from_sim no)
+		(in_bom yes)
+		(on_board yes)
+		(dnp no)
+		(fields_autoplaced yes)
+		(stroke
+			(width 0.1524)
+			(type solid)
+		)
+		(fill
+			(color 0 0 0 0.0000)
+		)
+		(property "Sheetname" "RS-485"
+			(at 38.1 67.8684 0)
+			(effects
+				(font
+					(size 1.27 1.27)
+				)
+				(justify left bottom)
+			)
+		)
+		(property "Sheetfile" "P1012202501-RS-485.kicad_sch"
+			(at 38.1 83.1346 0)
+			(effects
+				(font
+					(size 1.27 1.27)
+				)
+				(justify left top)
+			)
+		)
+		(instances
+			(project "P1012202501-Cover Sheet"
+				(path "/27f0531a-0a2b-4c68-af50-4332bf165b5a"
+					(page "4")
+				)
+			)
 		)
 	)

Commit message: Added new content from stream.
Other:
- added sheet Control Inputs (P1012202501-Control Inputs.kicad_sch)
- added sheet Limit Switches (P1012202501-Limit Switches.kicad_sch)
Changed lines of the file:
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@@
+	)
+	(sheet
+		(at 38.1 91.44)
+		(size 13.97 13.97)
+		(exclude_from_sim no)
+		(in_bom yes)
+		(on_board yes)
+		(dnp no)
+		(fields_autoplaced yes)
+		(stroke
+			(width 0.1524)
+			(type solid)
+		)
+		(fill
+			(color 0 0 0 0.0000)
+		)
+		(property "Sheetname" "Limit Switches"
+			(at 38.1 90.7284 0)
+			(effects
+				(font
+					(size 1.27 1.27)
+				)
+				(justify left bottom)
+			)
+		)
+		(property "Sheetfile" "P1012202501-Limit Switches.kicad_sch"
+			(at 38.1 105.9946 0)
+			(effects
+				(font
+					(size 1.27 1.27)
+				)
+				(justify left top)
+			)
+		)
+		(instances
+			(project "P1012202501-Cover Sheet"
+				(path "/27f0531a-0a2b-4c68-af50-4332bf165b5a"
+					(page "5")
+				)
+			)
+		)
 	)
 	(sheet
@@
 				)
 			)
+		)
+	)
+	(sheet
+		(at 38.1 115.57)
+		(size 13.97 13.97)
+		(exclude_from_sim no)
+		(in_bom yes)
+		(on_board yes)
+		(dnp no)
+		(fields_autoplaced yes)
+		(stroke
+			(width 0.1524)
+			(type solid)
+		)
+		(fill
+			(color 0 0 0 0.0000)
+		)
+		(property "Sheetname" "Control Inputs"
+			(at 38.1 114.8584 0)
+			(effects
+				(font
+					(size 1.27 1.27)
+				)
+				(justify left bottom)
+			)
+		)
+		(property "Sheetfile" "P1012202501-Control Inputs.kicad_sch"
+			(at 38.1 130.1246 0)
+			(effects
+				(font
+					(size 1.27 1.27)
+				)
+				(justify left top)
+			)
+		)
+		(instances
+			(project "P1012202501-Cover Sheet"
+				(path "/27f0531a-0a2b-4c68-af50-4332bf165b5a"
+					(page "6")
+				)
+			)

Commit message: Adding new content from stream.
Other:
- added sheet USB UART (P1012202501-USB UART.kicad_sch)
Changed lines of the file:
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@@
+		)
+	)
+	(sheet
+		(at 38.1 139.7)
+		(size 13.97 13.97)
+		(exclude_from_sim no)
+		(in_bom yes)
+		(on_board yes)
+		(dnp no)
+		(fields_autoplaced yes)
+		(stroke
+			(width 0.1524)
+			(type solid)
+		)
+		(fill
+			(color 0 0 0 0.0000)
+		)
+		(property "Sheetname" "USB UART"
+			(at 38.1 138.9884 0)
+			(effects
+				(font
+					(size 1.27 1.27)
+				)
+				(justify left bottom)
+			)
+		)
+		(property "Sheetfile" "P1012202501-USB UART.kicad_sch"
+			(at 38.1 154.2546 0)
+			(effects
+				(font
+					(size 1.27 1.27)
+				)
+				(justify left top)
+			)
+		)
+		(instances
+			(project "P1012202501-Cover Sheet"
+				(path "/27f0531a-0a2b-4c68-af50-4332bf165b5a"
+					(page "7")
+				)
+			)
 		)
 	)

Commit message: Added new content from stream.
Other:
- added sheet Stepper Driver (P1012202501-Stepper Driver.kicad_sch)
Changed lines of the file:
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@@
+	)
+	(sheet
+		(at 96.52 25.4)
+		(size 13.97 13.97)
+		(exclude_from_sim no)
+		(in_bom yes)
+		(on_board yes)
+		(dnp no)
+		(fields_autoplaced yes)
+		(stroke
+			(width 0.1524)
+			(type solid)
+		)
+		(fill
+			(color 0 0 0 0.0000)
+		)
+		(property "Sheetname" "Stepper Driver"
+			(at 96.52 24.6884 0)
+			(effects
+				(font
+					(size 1.27 1.27)
+				)
+				(justify left bottom)
+			)
+		)
+		(property "Sheetfile" "P1012202501-Stepper Driver.kicad_sch"
+			(at 96.52 39.9546 0)
+			(effects
+				(font
+					(size 1.27 1.27)
+				)
+				(justify left top)
+			)
+		)
+		(instances
+			(project "P1012202501-Cover Sheet"
+				(path "/27f0531a-0a2b-4c68-af50-4332bf165b5a"
+					(page "8")
+				)
+			)
+		)
 	)
 	(sheet

Commit message: Adding new materials from stream.
Parts:
- added FID1, FID2, FID3, FID4, FID5, FID6: ~, symbol COMPONENTS:FID1.0x1.5mmROUND
Other:
- note added: "FIDUCIALS"
