File: _Projects/P1012202501-ESP32_Stepper_Controller/Hardware/P1012202501-ESP32_Stepper_Controller/P1012202501-ESP32_Stepper_Controller.kicad_pcb (KiCad board)
At the start: 2 copper layers, 120 x 85.5 mm, 126 parts, among them CN1 KPTBP04R1-500-02BE, CN2 KPTBP04R1-500-03BE, CN3 KPTBP04R1-500-04BE, CN4 KPTBP04R1-500-04BE, CN5 KUSB4105-GF-A, CN6 KHS4B-PH-SM4-TB(LF)(SN), CN7 KPTBP04R1-500-04BE, IC1 PMAP63203WU-7, IC2 PMAP63205WU-7, IC3 ESP32-WROOM-32UE-N16, IC4 USP485REN-L_TR, IC5 UCP2102C-A01-GQFN28, IC6 UDRV8825PWPR, J1 KH22-28-5021, J2 KH22-28-5021, J3 KH22-28-5021, Q1 QTCMT1600T3, Q2 QTCMT1600T3, Q3 QTCMT1600T3, Q4 QTCMT1600T3, Q5 QTCMT1600T3, Q6 QTCMT1600T3, Q7 QBC847BDW1T1G

Commit message: Added new content and changes from stream.
Parts:
- moved CN4 272.9 mm to (81.5, 107.5), turned to -90 degrees
- moved CN6 265.2 mm to (110.8, 115.3)
- moved D3 259.4 mm to (91.0, 68.5), turned to 180 degrees
- moved IC3 256.8 mm to (132.4, 134.4)
- moved CN3 253.2 mm to (81.5, 87.0), turned to -90 degrees
- moved FID3 248.4 mm to (81.2, 43.8)
- moved C1 246.0 mm to (100.5, 70.5), turned to -90 degrees
- moved MH2 245.8 mm to (76.0, 57.5)
- moved C3 245.5 mm to (103.0, 70.5), turned to -90 degrees
- moved CN1 243.9 mm to (81.5, 68.5), turned to -90 degrees
- moved C2 242.9 mm to (100.5, 85.5), turned to -90 degrees
- moved IC2 242.9 mm to (107.0, 81.5), turned to -90 degrees
- moved IC1 242.4 mm to (107.0, 66.5), turned to -90 degrees
- moved C4 242.1 mm to (103.0, 85.5), turned to -90 degrees
- moved MH1 240.8 mm to (76.0, 130.5)
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Connections:
- CN7 pad 1: Net-(IC6-BOUT1) -> Net-(IC6-AOUT1)
- CN7 pad 2: Net-(IC6-BOUT2) -> Net-(IC6-AOUT2)
- CN7 pad 3: Net-(IC6-AOUT2) -> Net-(IC6-BOUT2)
- CN7 pad 4: Net-(IC6-AOUT1) -> Net-(IC6-BOUT1)
Other:
- copper layers 2 -> 6
- board text added: "+"
- board text added: "-"
- board text added: "3V OK"
- board text added: "5V OK"
- board text added: "COM"
- board text added: "CTL1"
- board text added: "CTL2"
- board text added: "CTL3"
- board text added: "DC"
- board text added: "LMT1"
- board text added: "LMT2"
- board text added: "LMT3"

Commit message: Added new content from the stream.
Parts:
- removed TP8, TP9: TP5010, CONNECTORS:5010
- C15, C16, C17, D4, FID4, FID5, FID6, IC4, R10, R11, R12, R13, R14, R15, R16, R17, R5, R6, R7, R8, R9: moved to B.Cu
- moved R12 289.3 mm to (76.0, 107.5), turned to 180 degrees
- moved R13 289.2 mm to (76.0, 112.5), turned to 180 degrees
- moved R14 289.1 mm to (76.0, 117.5), turned to 180 degrees
- moved R15 279.1 mm to (92.0, 108.0), turned to 180 degrees
- moved R16 278.6 mm to (92.0, 113.5), turned to 180 degrees
- moved R17 278.0 mm to (92.0, 119.5), turned to 180 degrees
- moved J3 277.8 mm to (91.0, 124.0)
- moved R6 271.4 mm to (76.0, 87.0), turned to 180 degrees
- moved R7 271.1 mm to (76.0, 92.0), turned to 180 degrees
- moved R8 270.8 mm to (76.0, 97.0), turned to 180 degrees
- moved Q4 265.9 mm to (92.0, 108.0)
- moved Q5 265.7 mm to (92.0, 113.5)
- moved Q6 265.5 mm to (92.0, 119.5)
- moved R9 262.8 mm to (92.0, 87.0), turned to 180 degrees
- moved R10 261.7 mm to (92.0, 92.5), turned to 180 degrees
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Other:
- board size 120 x 85.5 mm -> 120 x 85 mm
- board text added: "A"
- board text added: "A-1"
- board text added: "A-2"
- board text added: "B"
- board text added: "B-1"
- board text added: "B-2"
- board text added: "GND"

Commit message: Added items from latest stream.
Parts:
- added D7: TVSCDSOT23-SM712, COMPONENTS:SOT-23-3, F.Cu at (137.8, 132.1)
- added R31: RC06031K0075AAA, COMPONENTS:RES-0603, F.Cu at (106.1, 130.2)
- C11, C18, C19, D5, D6, Q7, R18, R19, R20, R21, R22, R26, R27, R3: moved to B.Cu
- moved LGO1 121.2 mm to (105.0, 55.1)
- moved R18 68.5 mm to (180.5, 117.5), turned to 180 degrees
- moved R22 68.1 mm to (170.0, 117.5)
- moved C21 67.3 mm to (180.0, 114.5), turned to 90 degrees
- moved R19 66.2 mm to (173.5, 115.5), turned to 90 degrees
- moved C20 64.5 mm to (178.5, 114.5), turned to 90 degrees
- moved D6 60.3 mm to (188.0, 119.5), turned to -90 degrees
- moved C19 59.8 mm to (175.0, 115.5), turned to 90 degrees
- moved C18 59.0 mm to (176.5, 115.5), turned to 90 degrees
- moved TP23 57.2 mm to (176.0, 128.0)
- moved Q7 53.7 mm to (134.0, 118.7), turned to 180 degrees
- moved R21 51.5 mm to (144.0, 118.9), turned to 180 degrees
- moved TP22 49.9 mm to (171.0, 128.0)
- moved D5 48.2 mm to (179.5, 124.5), turned to -90 degrees
- moved R20 46.8 mm to (138.5, 119.6), turned to 180 degrees
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Connections:
- C20 pad 1: +3.3V -> +3V3
- C21 pad 1: +3.3V -> +3V3
- IC5 pad 6: +3.3V -> +3V3
- IC5 pad 7: +3.3V -> +3V3
- Q1 pad 4: +3.3V -> +3V3
- Q2 pad 4: +3.3V -> +3V3
- Q3 pad 4: +3.3V -> +3V3
- Q4 pad 4: +3.3V -> +3V3
- Q5 pad 4: +3.3V -> +3V3
- Q6 pad 4: +3.3V -> +3V3
- R22 pad 1: +3.3V -> +3V3
Routing:
- net +24V: track 0.00 -> 125.8 mm
- net Net-(D3-A): track 0.00 -> 7.45 mm
- net GND: vias 0 -> 3
- added copper zone on In1.Cu, net +3V3
- added copper zone on F.Cu, net GND
- added copper zone on In4.Cu, net GND
Other:
- board text added: "P1012202501-PCB-01"

Commit message: Added updated items from recent stream.
Parts:
- moved C26 4.41 mm to (168.0, 78.5), turned to 90 degrees
- moved C25 1.65 mm to (173.0, 78.5)
- moved R25 1.26 mm to (171.0, 78.5)
- moved C23 0.36 mm to (170.5, 67.0)
- moved C24 0.36 mm to (170.5, 68.5)
- moved R29 0.20 mm to (153.5, 67.5)
- moved C27 0.10 mm to (160.0, 67.5)
Routing:
- net /Control Inputs/INPUT_C: track 0.00 -> 40.5 mm
- net /Limit Switches/LMT_C: track 0.00 -> 37.4 mm
- net +24V: track 125.8 -> 155.6 mm, vias 0 -> 2
- net GND: track 0.00 -> 23.5 mm, vias 3 -> 50
- net +3V3: track 0.00 -> 23.5 mm, vias 0 -> 11
- net Net-(Q6-A): track 0.00 -> 19.4 mm, vias 0 -> 1
- net Net-(Q1-A): track 0.00 -> 18.3 mm, vias 0 -> 1
- net Net-(Q3-A): track 0.00 -> 18.0 mm, vias 0 -> 1
- net Net-(Q5-A): track 0.00 -> 17.8 mm, vias 0 -> 1
- net Net-(Q2-A): track 0.00 -> 17.7 mm, vias 0 -> 1
- net LIMIT_1: track 0.00 -> 17.5 mm, vias 0 -> 1
- net Net-(Q4-A): track 0.00 -> 17.5 mm, vias 0 -> 1
- net Net-(IC6-BOUT1): track 0.00 -> 17.2 mm
- net LIMIT_3: track 0.00 -> 17.1 mm, vias 0 -> 1
- net LIMIT_2: track 0.00 -> 17.0 mm, vias 0 -> 1
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- added copper zone on F.Cu, net +3V3
- added copper zone on F.Cu, net +5V
- added copper zone on F.Cu, net Net-(IC1-SW)
- added copper zone on F.Cu, net Net-(IC2-SW)

Commit message: Added new content from stream.
Parts:
- C11, R3: moved to F.Cu
- moved C14 16.9 mm to (150.5, 102.5), turned to 90 degrees
- moved C13 15.2 mm to (148.5, 102.5), turned to 90 degrees
- moved C12 14.0 mm to (146.5, 102.5), turned to 90 degrees
- moved R3 10.3 mm to (144.3, 102.5), turned to -90 degrees
- moved C11 8.84 mm to (142.0, 102.5), turned to 90 degrees
- moved D4 1.00 mm to (186.0, 105.5), turned to 0 degrees
- moved R27 0.36 mm to (171.0, 72.5), turned to 180 degrees
- moved R26 0.32 mm to (171.0, 74.5), turned to 180 degrees
- moved Q7 0.20 mm to (134.0, 118.5)
Routing:
- net +5V: track 16.3 -> 82.0 mm, vias 0 -> 6
- net VBUS: track 0.00 -> 34.3 mm, vias 0 -> 2
- net Net-(IC4-A): track 0.00 -> 32.0 mm, vias 0 -> 1
- net /USB UART/USB_D_P: track 0.00 -> 25.3 mm, vias 0 -> 1
- net /USB UART/USB_D_N: track 0.00 -> 22.7 mm, vias 0 -> 2
- net Net-(IC4-B): track 0.00 -> 21.3 mm
- net GND: track 23.5 -> 40.1 mm, vias 50 -> 88
- net Net-(IC6-AVREF): track 5.62 -> 21.2 mm
- net 485_RX: track 0.00 -> 15.3 mm
- net 485_DIR: track 0.00 -> 13.7 mm
- net Net-(IC5-VBUS): track 0.00 -> 10.7 mm, vias 0 -> 1
- net Net-(IC6-ISENB): track 0.00 -> 9.71 mm, vias 0 -> 1
- net Net-(IC6-ISENA): track 0.00 -> 9.55 mm, vias 0 -> 1
- net 485_TX: track 0.00 -> 8.21 mm
- net Net-(IC5-RSTB): track 0.00 -> 7.20 mm, vias 0 -> 1
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- added copper zone on B.Cu, net +5V
- added copper zone on B.Cu, net GND

Commit message: Added new content from latest stream.
Parts:
- added D8: TVSCDSOT23-SM712, COMPONENTS:SOT-23-3, B.Cu at (118.0, 114.5)
- added J4: KH68001-406HLF, CONNECTORS:6x1HDR2.54mm, F.Cu at (123.0, 105.5)
- IC4: value USP485REN-L_TR -> USP3485CN-L/TR
- R23, R24, R30, R4: moved to B.Cu
- moved R31 80.8 mm to (141.2, 57.5)
- moved CN6 78.3 mm to (146.0, 61.5), turned to 180 degrees
- moved TP19 66.4 mm to (157.0, 105.5)
- moved TP21 58.5 mm to (157.0, 110.5)
- moved TP18 55.2 mm to (157.0, 115.5)
- moved TP20 44.2 mm to (157.0, 120.5)
- moved R30 28.2 mm to (137.5, 121.5), turned to -90 degrees
- moved R4 24.4 mm to (128.0, 124.5)
- moved S2 23.1 mm to (151.0, 131.5), turned to 180 degrees
- moved S1 18.6 mm to (128.0, 131.5), turned to 180 degrees
- moved Q7 15.0 mm to (148.5, 114.5), turned to -90 degrees
- moved R20 14.0 mm to (151.5, 114.5), turned to -90 degrees
- moved R24 13.0 mm to (133.0, 111.0), turned to 180 degrees
- moved R23 6.15 mm to (132.5, 103.5), turned to -90 degrees
- moved R21 4.65 mm to (145.5, 114.5), turned to -90 degrees
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Connections:
- C15 pad 1: +5V -> +3V3
- C16 pad 1: +5V -> +3V3
- C17 pad 1: +5V -> +3V3
- CN6 pad 5: (no net) -> GND
- CN6 pad 6: (no net) -> GND
- IC3 pad 31: UART_RX -> /ESP32/UART_RX
- IC3 pad 33: UART_TX -> /ESP32/UART_TX
- IC4 pad 8: +5V -> +3V3
Routing:
- net ESP_EN: track 6.19 -> 64.6 mm, vias 0 -> 2
- net BOOT_MODE: track 0.00 -> 57.9 mm, vias 0 -> 1
- net /USB UART/DTR: track 0.00 -> 57.1 mm, vias 0 -> 1
- net ESP_RX: track 0.00 -> 41.2 mm, vias 0 -> 2
- net /USB UART/RTS: track 0.00 -> 37.7 mm, vias 0 -> 1
- net ESP_TX: track 0.00 -> 37.6 mm, vias 0 -> 2
- net +5V: track 82.0 -> 52.6 mm, vias 6 -> 0
- net +3V3: track 25.7 -> 33.0 mm, vias 22 -> 31
- net STP_RESET: track 0.00 -> 6.65 mm, vias 0 -> 1
- net /ESP32/UART_RX: track 0.00 -> 6.18 mm
- net /ESP32/UART_TX: track 0.00 -> 6.09 mm
- net STP_FLT: track 0.00 -> 4.93 mm, vias 0 -> 1
- net Net-(Q7-B1): track 0.00 -> 4.13 mm
- net FAN_TACH: track 0.00 -> 4.01 mm
- net Net-(Q7-B2): track 0.00 -> 3.99 mm
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- added copper zone on B.Cu, net +3V3
- removed copper zone on B.Cu, net +5V
Other:
- board text added: "BOOT"
- board text added: "DEBUG INTERFACE"
- board text added: "ENABLE"

Commit message: Added latest content from stream.
Parts:
- added C28: CC0603104050AAAX7R, COMPONENTS:CAP-0603, F.Cu at (160.0, 83.5)
- added C29: CC0603226010AABX5R, COMPONENTS:CAP-0603, F.Cu at (160.0, 85.0)
- added D9: DLLS R976-NR-1, COMPONENTS:LED-0805, F.Cu at (133.0, 95.5)
- added IC7: UTMP36GRTZ-REEL7, COMPONENTS:SOT-23-5, F.Cu at (165.0, 83.5)
- added R32: RC0603330075AAA, COMPONENTS:RES-0603, F.Cu at (133.0, 98.5)
Connections:
- IC3 pad 24: unconnected-(IC3-IO2-Pad24) -> TEMP_SENSE
- IC3 pad 26: unconnected-(IC3-IO4-Pad26) -> Net-(IC3-IO4)
Routing:
- net TEMP_SENSE: track 0.00 -> 85.0 mm, vias 0 -> 2
- net STP_FLT: track 4.93 -> 80.5 mm, vias 1 -> 2
- net FAN_PWM: track 0.00 -> 70.4 mm, vias 0 -> 2
- net STP_MS0: track 0.00 -> 68.6 mm, vias 0 -> 2
- net STP_DIR: track 0.00 -> 67.3 mm, vias 0 -> 2
- net STP_MS1: track 0.00 -> 66.3 mm, vias 0 -> 2
- net FAN_TACH: track 4.01 -> 69.7 mm, vias 0 -> 2
- net STP_RESET: track 6.65 -> 71.4 mm, vias 1 -> 2
- net STP_MS2: track 0.00 -> 63.8 mm, vias 0 -> 2
- net INPUT_3: track 12.8 -> 68.9 mm, vias 1 -> 2
- net INPUT_2: track 13.6 -> 66.5 mm, vias 1 -> 2
- net STP_STEP: track 0.00 -> 52.9 mm, vias 0 -> 2
- net STP_ENABLE: track 2.56 -> 53.7 mm, vias 1 -> 2
- net INPUT_1: track 13.7 -> 63.8 mm, vias 1 -> 2
- net LIMIT_3: track 17.1 -> 65.5 mm, vias 1 -> 2
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Other:
- board text added: "STATUS"

Commit message: Added new content from stream.
Parts:
- moved TP7 25.7 mm to (154.0, 96.5)
Routing:
- net GND: vias 116 -> 119
