File: _Projects/P1012202501-ESP32_Stepper_Controller/Hardware/P1012202501-ESP32_Stepper_Controller/P1012202501-ESP32_Stepper_Controller.kicad_pcb (KiCad board)
At the start: 6 copper layers, 120 x 85 mm, 133 parts, among them CN1 KPTBP04R1-500-02BE, CN2 KPTBP04R1-500-03BE, CN3 KPTBP04R1-500-04BE, CN4 KPTBP04R1-500-04BE, CN5 KUSB4105-GF-A, CN6 KHS4B-PH-SM4-TB(LF)(SN), CN7 KPTBP04R1-500-04BE, IC1 PMAP63203WU-7, IC2 PMAP63205WU-7, IC3 ESP32-WROOM-32UE-N16, IC4 USP3485CN-L/TR, IC5 UCP2102C-A01-GQFN28, IC6 UDRV8825PWPR, IC7 UTMP36GRTZ-REEL7, J1 KH22-28-5021, J2 KH22-28-5021, J3 KH22-28-5021, J4 KH68001-406HLF, Q1 QTCMT1600T3, Q2 QTCMT1600T3, Q3 QTCMT1600T3, Q4 QTCMT1600T3, Q5 QTCMT1600T3, Q6 QTCMT1600T3, Q7 QBC847BDW1T1G

Commit message: Added new content from stream.
Other:
- board text added: "P1012202501-PCB-02"
- board text removed: "P1012202501-PCB-01"
Changed lines of the file:
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@@
 		(layer "Edge.Cuts")
 	)
-	(gr_text "P1012202501-PCB-01"
+	(gr_text "P1012202501-PCB-02"
 		(at 147 54.5 0)
 		(layer "B.Cu")

Commit message: Added new items from streams.
Parts:
- added C30: CC0603104050AAAX7R, COMPONENTS:CAP-0603, F.Cu at (126.0, 120.5)
- added TP26: TP5010, CONNECTORS:5010, F.Cu at (172.0, 83.5)
- added TP27: TP5010, CONNECTORS:5010, F.Cu at (147.0, 82.5)
- added TP28: TP5010, CONNECTORS:5010, F.Cu at (152.0, 82.5)
- added TP29: TP5010, CONNECTORS:5010, F.Cu at (147.0, 89.5)
- added TP30: TP5010, CONNECTORS:5010, F.Cu at (152.0, 89.5)
- added TP31: TP5010, CONNECTORS:5010, F.Cu at (162.0, 89.5)
- added TP32: TP5010, CONNECTORS:5010, F.Cu at (167.0, 89.5)
- added TP33: TP5010, CONNECTORS:5010, F.Cu at (172.0, 89.5)
- added TP34: TP5010, CONNECTORS:5010, F.Cu at (157.0, 89.5)
- added TP35: TP5010, CONNECTORS:5010, F.Cu at (129.0, 58.0)
- added TP36: TP5010, CONNECTORS:5010, F.Cu at (134.0, 58.0)
- added TP8: TP5010, CONNECTORS:5010, F.Cu at (165.0, 110.5)
- added TP9: TP5010, CONNECTORS:5010, F.Cu at (165.0, 115.5)
- R10, R11, R15, R16, R17, R9: value RC06010K2075AAA -> RC060310K2075AAA
- moved CN1 2.00 mm to (79.5, 68.5)
- moved CN2 2.00 mm to (182.5, 108.5)
- moved CN3 2.00 mm to (79.5, 87.0)
- moved CN4 2.00 mm to (79.5, 107.5)
- moved CN7 2.00 mm to (182.5, 80.5)
- moved R5 2.00 mm to (187.0, 99.5)
- moved R12 1.00 mm to (75.0, 107.5)
- moved R13 1.00 mm to (75.0, 112.5)
- moved R14 1.00 mm to (75.0, 117.5)
- moved R6 1.00 mm to (75.0, 87.0)
- moved R7 1.00 mm to (75.0, 92.0)
- moved R8 1.00 mm to (75.0, 97.0)
- moved D4 0.50 mm to (186.5, 105.5)
Connections:
- CN6 pad 5: GND -> (no net)
- CN6 pad 6: GND -> (no net)
Routing:
- net STP_MS2: track 63.8 -> 105.7 mm
- net STP_MS1: track 66.3 -> 106.1 mm
- net STP_MS0: track 68.6 -> 105.8 mm
- net STP_RESET: track 71.4 -> 105.3 mm
- net STP_FLT: track 80.5 -> 106.4 mm
- net STP_DIR: track 67.3 -> 93.0 mm
- net STP_STEP: track 52.9 -> 73.9 mm
- net ESP_RX: track 41.2 -> 57.5 mm
- net FAN_TACH: track 69.7 -> 84.3 mm
- net FAN_PWM: track 70.4 -> 83.3 mm
- net TEMP_SENSE: track 85.0 -> 96.4 mm
- net STP_ENABLE: track 53.7 -> 65.2 mm
- net ESP_TX: track 37.6 -> 48.5 mm
- net Net-(IC6-BOUT1): track 17.2 -> 21.2 mm
- net Net-(IC6-AOUT2): track 15.3 -> 17.3 mm
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
Commit message: Adding new items from recent streams.
Parts:
- moved C30 19.7 mm to (136.0, 103.5), turned to 180 degrees
Connections:
- IC3 pad 24: TEMP_SENSE -> INPUT_1
- IC3 pad 8: INPUT_1 -> TEMP_SENSE
Routing:
- net TEMP_SENSE: track 96.4 -> 64.6 mm
- net INPUT_1: track 63.8 -> 60.0 mm, vias 2 -> 1
