File: _Projects/P1012202501-ESP32_Stepper_Controller/Hardware/P1012202501-ESP32_Stepper_Controller/P1012202501-Power Supplies.kicad_sch (KiCad schematic)
At the start: 14 parts, among them IC1 PMAP63203WU-7, IC2 PMAP63205WU-7

Commit message: Pushing updated content.
Parts:
- C1, C2, C6, C7: Val (none) -> 10µF, 50V, 1206
- C10, C4, C5, C9: Val (none) -> 22µF, 25V, 1210
- C3, C8: Val (none) -> 0.1µF, 50V, 0603
- IC1: footprint COMPONENTS:AP63203WU7 -> COMPONENTS:TSOT-26-6
- L1, L2: Val (none) -> 2.2µH, 2.3A
Other:
- removed sheet ESP32
- moved on the sheet: C1, C10, C2, C3, C4, C5, C6, C7, C8, C9, IC1, IC2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

Commit message: Adding new content from stream.
Parts:
- added D2: DSSS26SHE3_B_H, COMPONENTS:SMA, symbol COMPONENTS:DSSS26SHE3_B_H
- added D3, D4: DLQ62702P5179, COMPONENTS:LED-0805, symbol COMPONENTS:DLQ62702P5179
- added J2: KP39522-0002, CONNECTORS:39522-0002, symbol CONNECTORS:KP39522-0002
- added R10: RC0603510075AAA, COMPONENTS:RES-0603, symbol COMPONENTS:RC0603510075AAA
- added R9: RC0603330075AAA, COMPONENTS:RES-0603, symbol COMPONENTS:RC0603330075AAA
- added TP1, TP2, TP3: TP5010, CONNECTORS:5010, symbol CONNECTORS:TP5010
Connections:
- net +24V: now also D2.1 (K)
- net +3V3: now also R9.1, TP1.1
- net +5V: now also R10.1, TP2.1
- net GND: now also D3.1 (K), D4.1 (K), J2.2, TP3.1
- new net: D3.2 (A), R9.2
- new net: D2.2 (A), J2.1
- new net: D4.2 (A), R10.2
Other:
- moved on the sheet: C1, C10, C2, C3, C4, C5, C6, C7, C8, C9, IC1, IC2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

Commit message: Adding content from latest stream.
Parts:
- renumbered J2 to CN2
Changed lines of the file:
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@@
 		(on_board yes)
 		(dnp no)
-		(property "Reference" "J2"
-			(at 24.892 24.13 0)
+		(property "Reference" "CN2"
+			(at 27.686 23.368 0)
 			(effects
 				(font
 					(size 1.27 1.27)
 				)
+				(justify left top)
 			)
 		)
 		(property "Value" "KP39522-0002"
-			(at 31.242 34.29 0)
+			(at 36.068 34.036 0)
 			(effects
 				(font
 					(size 1.27 1.27)
 				)
+				(justify left top)
 			)
 		)
@@
 		)
 		(property "Mate" "39520-0002"
-			(at 30.734 36.576 0)
+			(at 28.448 36.83 0)
 			(show_name yes)
 			(effects
@@
 			(project ""
 				(path "/27f0531a-0a2b-4c68-af50-4332bf165b5a/d737bb1a-43fc-4186-97c6-d6ed9cc0125d"
-					(reference "J2")
+					(reference "CN2")
 					(unit 1)
 				)

Commit message: Adding new content from stream.
Parts:
- removed CN2: KP39522-0002, CONNECTORS:39522-0002, symbol CONNECTORS:KP39522-0002
- added CN2: KPTBP04R1-500-02BE, CONNECTORS:TBP04R1-500-02BE, symbol CONNECTORS:KPTBP04R1-500-02BE
Connections:
- net GND: now also CN2.2
- net at D2.2 (A): now also CN2.1
Changed lines of the file:
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@@
 	)
 	(symbol
-		(lib_id "CONNECTORS:KP39522-0002")
+		(lib_id "CONNECTORS:KPTBP04R1-500-02BE")
 		(at 39.37 27.94 0)
 		(mirror y)
@@
 		(on_board yes)
 		(dnp no)
+		(fields_autoplaced yes)
 		(property "Reference" "CN2"
-			(at 27.686 23.368 0)
+			(at 29.21 17.78 0)
+			(effects
+				(font
+					(size 1.524 1.524)
+				)
+			)
+		)
+		(property "Value" "KPTBP04R1-500-02BE"
+			(at 29.21 20.32 0)
+			(effects
+				(font
+					(size 1.524 1.524)
+				)
+			)
+		)
+		(property "Footprint" "CONNECTORS:TBP04R1-500-02BE"
+			(at 48.514 21.082 0)
 			(effects
 				(font
 					(size 1.27 1.27)
+					(italic yes)
 				)
-				(justify left top)
-			)
-		)
-		(property "Value" "KP39522-0002"
-			(at 36.068 34.036 0)
-			(effects
-				(font
-					(size 1.27 1.27)
-				)
-				(justify left top)
-			)
-		)
-		(property "Footprint" "CONNECTORS:39522-0002"
-			(at 22.86 122.86 0)
-			(effects
-				(font
-					(size 1.27 1.27)
-				)
-				(justify left top)
 				(hide yes)
 			)
 		)
 		(property "Datasheet" ""
-			(at 22.86 222.86 0)
+			(at 39.116 37.846 0)
 			(effects
 				(font
 					(size 1.27 1.27)
+					(italic yes)
 				)
-				(justify left top)
 				(hide yes)
 			)
 		)
-		(property "Description" "Connector, Pluggable, 2 Circuit, 1 Row, Right Angle, Through Hole, 5.0mm Pitch, 300V @ 18A, RoHS"
+		(property "Description" "Connector, Pluggable, 2 Circuit, 1 Row, Right Angle, Through Hole, 5.0mm Pitch, 300V @ 15A, RoHS, Blue"
 			(at 39.37 27.94 0)
 			(effects
@@
 			)
 		)
-		(property "Manufacturer 1" "Molex"
+		(property "Manufacturer 1" "Same Sky"
 			(at 39.37 27.94 0)
 			(effects
@@
 			)
 		)
-		(property "Manufacturer 1 P/N" "39522-0002"
+		(property "Manufacturer 1 P/N" "TBP04R1-500-02BE"
 			(at 39.37 27.94 0)
 			(effects
@@
 			)
 		)
-		(property "Vendor 1a P/N" "538-39522-0002"
+		(property "Vendor 1a P/N" "179-TBP04R1-500-02BE"
 			(at 39.37 27.94 0)
 			(effects
@@
 			)
 		)
-		(property "Vendor 1a Cost LV" "0.31"
+		(property "Vendor 1a Cost LV" "0.33"
 			(at 39.37 27.94 0)
 			(effects
@@
 			)
 		)
-		(property "Vendor 1a Cost HV" "0.308"
+		(property "Vendor 1a Cost HV" "0.128"
 			(at 39.37 27.94 0)
 			(effects
@@
 			)
 		)
-		(property "Mate" "39520-0002"
-			(at 28.448 36.83 0)
+		(property "Mate" "TBP04P1-500-02BE"
+			(at 29.21 22.86 0)
 			(show_name yes)
 			(effects
@@
 			)
 		)
+		(pin "1"
+		)
 		(pin "2"
 		)
-		(pin "1"
-		)
 		(instances

Commit message: Added new items from stream.
Parts:
- renumbered C6 to C2, C2 to C3, C7 to C4, C3 to C5, C8 to C6, C4 to C7, C9 to C8, C5 to C9, CN2 to CN1, D3 to D1, D4 to D2, D2 to D3, R9 to R1, R10 to R2

Commit message: Added new content from stream.
Other:
- note added: "2"
Changed lines of the file:
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@@
 	(generator_version "9.0")
 	(paper "A4")
+	(text "2"
+		(exclude_from_sim no)
+		(at 268.986 193.548 0)
+		(effects
+			(font
+				(size 1.27 1.27)
+			)
+		)
+	)
 	(text "Power Supplies"
 		(exclude_from_sim yes)
