File: _Projects/P1012202501-ESP32_Stepper_Controller/Hardware/P1012202501-ESP32_Stepper_Controller/P1012202501-RS-485.kicad_sch (KiCad schematic)
At the start: 5 parts, among them IC4 USP485REN-L_TR

Commit message: Added new content from stream.
Parts:
- added J1: KH22-28-5021, CONNECTORS:2x1HDR2.54mm, symbol CONNECTORS:KH22-28-5021
- added R2: RC0805121150AAB, COMPONENTS:RES-0805, symbol COMPONENTS:RC0805121150AAB
Connections:
- net 485_A: now also J1.2
- net 485_B: now also R2.1
- new net: J1.1, R2.2
Other:
- moved on the sheet: D1

Commit message: Adding content from latest stream.
Parts:
- added CN1: KP39522-0003, CONNECTORS:39522-0003, symbol CONNECTORS:KP39522-0003
- added TP4, TP5, TP6, TP7, TP8, TP9: TP5010, CONNECTORS:5010, symbol CONNECTORS:TP5010
Connections:
- net 485_DIR: now also TP7.1
- net 485_RX: now also TP6.1
- net 485_TX: now also TP8.1
- net GND: now also CN1.3, TP9.1
- net 485_A: no longer names the net of D1.1, IC4.6 (A), J1.2
- net 485_A: now also CN1.2, TP5.1
- net 485_B: no longer names the net of D1.2, IC4.7 (B), R2.1
- net 485_B: now also CN1.1, TP4.1
Other:
- moved on the sheet: C15, C16, C17, D1, IC4, J1, R2

Commit message: Adding new content from stream.
Parts:
- removed CN1: KP39522-0003, CONNECTORS:39522-0003, symbol CONNECTORS:KP39522-0003
- added CN1: KPTBP04R1-500-03BE, CONNECTORS:TBP04R1-500-03BE, symbol CONNECTORS:KPTBP04R1-500-03BE
Connections:
- net GND: now also CN1.3
- net at D1.2, IC4.7 (B), R2.1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: now also CN1.1
- net at D1.1, IC4.6 (A), J1.2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: now also CN1.2
Changed lines of the file:
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@@
 	)
 	(symbol
-		(lib_id "CONNECTORS:KP39522-0003")
+		(lib_id "CONNECTORS:KPTBP04R1-500-03BE")
 		(at 224.79 78.74 0)
 		(unit 1)
@@
 			)
 		)
-		(property "Value" "KP39522-0003"
+		(property "Value" "KPTBP04R1-500-03BE"
 			(at 241.3 81.2799 0)
 			(effects
@@
 			)
 		)
-		(property "Footprint" "CONNECTORS:39522-0003"
+		(property "Footprint" "CONNECTORS:TBP04R1-500-03BE"
 			(at 215.646 71.882 0)
 			(effects
@@
 			)
 		)
-		(property "Description" "Connector, Pluggable, 3 Circuit, 1 Row, Right Angle, Through Hole, 5.0mm Pitch, 300V @ 15A, RoHS"
+		(property "Description" "Connector, Pluggable, 4 Circuit, 1 Row, Right Angle, Through Hole, 5.0mm Pitch, 300V @ 15A, RoHS, Blue"
 			(at 224.79 78.74 0)
 			(effects
@@
 			)
 		)
-		(property "Manufacturer 1" "Molex"
+		(property "Manufacturer 1" "Same Sky"
 			(at 224.79 78.74 0)
 			(effects
@@
 			)
 		)
-		(property "Manufacturer 1 P/N" "39522-0003"
+		(property "Manufacturer 1 P/N" "TBP04R1-500-03BE"
 			(at 224.79 78.74 0)
 			(effects
@@
 			)
 		)
-		(property "Vendor 1a P/N" "538-39522-0003"
+		(property "Vendor 1a P/N" "179-TBP04R1-500-03BE"
 			(at 224.79 78.74 0)
 			(effects
@@
 			)
 		)
-		(property "Vendor 1a Cost LV" "0.52"
+		(property "Vendor 1a Cost LV" "0.48"
 			(at 224.79 78.74 0)
 			(effects
@@
 			)
 		)
-		(property "Vendor 1a Cost HV" "0.471"
+		(property "Vendor 1a Cost HV" "0.189"
 			(at 224.79 78.74 0)
 			(effects
@@
 			)
 		)
-		(property "Mate" "39520-0003"
+		(property "Mate" "TBP04P1-500-03BE"
 			(at 241.3 83.8199 0)
 			(show_name yes)
@@
 			)
 		)
-		(pin "2"
-		)
 		(pin "1"
 		)
 		(pin "3"
 		)
+		(pin "2"
+		)
 		(instances

Commit message: Added new items from stream.
Parts:
- renumbered C17 to C15, C15 to C17, CN1 to CN2, D1 to D4, R2 to R5, TP6 to TP4, TP7 to TP5, TP8 to TP6, TP9 to TP7, TP4 to TP8, TP5 to TP9
Changed lines of the file:
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@@
 		(on_board yes)
 		(dnp no)
-		(property "Reference" "TP8"
+		(property "Reference" "TP6"
 			(at 75.946 113.284 90)
 			(effects
@@
 			(project ""
 				(path "/27f0531a-0a2b-4c68-af50-4332bf165b5a/f7d1483b-b2e1-4d1b-a579-3453a4da28ca"
-					(reference "TP8")
+					(reference "TP6")
 					(unit 1)
 				)
@@
 		(on_board yes)
 		(dnp no)
-		(property "Reference" "TP7"
+		(property "Reference" "TP5"
 			(at 65.786 113.284 90)
 			(effects
@@
 			(project ""
 				(path "/27f0531a-0a2b-4c68-af50-4332bf165b5a/f7d1483b-b2e1-4d1b-a579-3453a4da28ca"
-					(reference "TP7")
+					(reference "TP5")
 					(unit 1)
 				)
@@
 		(dnp no)
 		(fields_autoplaced yes)
-		(property "Reference" "CN1"
+		(property "Reference" "CN2"
 			(at 241.3 78.7399 0)
 			(effects
@@
 			(project ""
 				(path "/27f0531a-0a2b-4c68-af50-4332bf165b5a/f7d1483b-b2e1-4d1b-a579-3453a4da28ca"
-					(reference "CN1")
+					(reference "CN2")
 					(unit 1)
 				)
@@
 		(dnp no)
 		(fields_autoplaced yes)
-		(property "Reference" "#PWR035"
+		(property "Reference" "#PWR031"
 			(at 223.52 96.52 0)
 			(effects
@@
 			(project "P1012202501-Cover Sheet"
 				(path "/27f0531a-0a2b-4c68-af50-4332bf165b5a/f7d1483b-b2e1-4d1b-a579-3453a4da28ca"
-					(reference "#PWR035")
+					(reference "#PWR031")
 					(unit 1)
 				)
@@
 		(dnp no)
 		(fields_autoplaced yes)
-		(property "Reference" "#PWR017"
+		(property "Reference" "#PWR029"
 			(at 120.65 93.98 0)
 			(effects
@@
 			(project ""
 				(path "/27f0531a-0a2b-4c68-af50-4332bf165b5a/f7d1483b-b2e1-4d1b-a579-3453a4da28ca"
-					(reference "#PWR017")
+					(reference "#PWR029")
 					(unit 1)
 				)
@@
 		(on_board yes)
 		(dnp no)
-		(property "Reference" "D1"
+		(property "Reference" "D4"
 			(at 169.164 111.76 0)
 			(effects
@@
 			(project ""
 				(path "/27f0531a-0a2b-4c68-af50-4332bf165b5a/f7d1483b-b2e1-4d1b-a579-3453a4da28ca"
-					(reference "D1")
+					(reference "D4")
 					(unit 1)
 				)
@@
 	)
 	(symbol
-		(lib_name "CC0805226025AABX5R_1")
 		(lib_id "COMPONENTS:CC0805226025AABX5R")
 		(at 101.6 45.72 270)
@@
 		(dnp no)
 		(fields_autoplaced yes)
-		(property "Reference" "TP5"
+		(property "Reference" "TP9"
 			(at 205.74 104.1399 0)
 			(effects
@@
 			(project ""
 				(path "/27f0531a-0a2b-4c68-af50-4332bf165b5a/f7d1483b-b2e1-4d1b-a579-3453a4da28ca"
-					(reference "TP5")
+					(reference "TP9")
 					(unit 1)
 				)
@@
 		(dnp no)
 		(fields_autoplaced yes)
-		(property "Reference" "#PWR036"
+		(property "Reference" "#PWR026"
 			(at 88.9 125.73 0)
 			(effects
@@
 			(project "P1012202501-Cover Sheet"
 				(path "/27f0531a-0a2b-4c68-af50-4332bf165b5a/f7d1483b-b2e1-4d1b-a579-3453a4da28ca"
-					(reference "#PWR036")
+					(reference "#PWR026")
 					(unit 1)
 				)
@@
 		(on_board yes)
 		(dnp no)
-		(property "Reference" "C17"
+		(property "Reference" "C15"
 			(at 91.186 50.038 90)
 			(effects
@@
 			(project ""
 				(path "/27f0531a-0a2b-4c68-af50-4332bf165b5a/f7d1483b-b2e1-4d1b-a579-3453a4da28ca"
-					(reference "C17")
+					(reference "C15")
 					(unit 1)
 				)
@@
 		(dnp no)
 		(fields_autoplaced yes)
-		(property "Reference" "#PWR019"
+		(property "Reference" "#PWR030"
 			(at 186.69 129.54 0)
 			(effects
@@
 			(project "P1012202501-Cover Sheet"
 				(path "/27f0531a-0a2b-4c68-af50-4332bf165b5a/f7d1483b-b2e1-4d1b-a579-3453a4da28ca"
-					(reference "#PWR019")
+					(reference "#PWR030")
 					(unit 1)
 				)
@@
 		(on_board yes)
 		(dnp no)
-		(property "Reference" "TP6"
+		(property "Reference" "TP4"
 			(at 55.372 113.284 90)
 			(effects
@@
 			(project ""
 				(path "/27f0531a-0a2b-4c68-af50-4332bf165b5a/f7d1483b-b2e1-4d1b-a579-3453a4da28ca"
-					(reference "TP6")
+					(reference "TP4")
 					(unit 1)
 				)
@@
 		(dnp no)
 		(fields_autoplaced yes)
-		(property "Reference" "#PWR013"
+		(property "Reference" "#PWR028"
 			(at 119.38 46.99 0)
 			(effects
@@
 			(project ""
 				(path "/27f0531a-0a2b-4c68-af50-4332bf165b5a/f7d1483b-b2e1-4d1b-a579-3453a4da28ca"
-					(reference "#PWR013")
+					(reference "#PWR028")
 					(unit 1)
 				)
@@
 		(dnp no)
 		(fields_autoplaced yes)
-		(property "Reference" "R2"
+		(property "Reference" "R5"
 			(at 168.91 66.0399 90)
 			(effects
@@
 			(project ""
 				(path "/27f0531a-0a2b-4c68-af50-4332bf165b5a/f7d1483b-b2e1-4d1b-a579-3453a4da28ca"
-					(reference "R2")
+					(reference "R5")
 					(unit 1)
 				)
@@
 		(dnp no)
 		(fields_autoplaced yes)
-		(property "Reference" "TP4"
+		(property "Reference" "TP8"
 			(at 205.74 48.2599 0)
 			(effects
@@
 			(project ""
 				(path "/27f0531a-0a2b-4c68-af50-4332bf165b5a/f7d1483b-b2e1-4d1b-a579-3453a4da28ca"
-					(reference "TP4")
+					(reference "TP8")
 					(unit 1)
 				)
@@
 		(on_board yes)
 		(dnp no)
-		(property "Reference" "TP9"
+		(property "Reference" "TP7"
 			(at 87.122 100.584 90)
 			(effects
@@
 			(project ""
 				(path "/27f0531a-0a2b-4c68-af50-4332bf165b5a/f7d1483b-b2e1-4d1b-a579-3453a4da28ca"
-					(reference "TP9")
+					(reference "TP7")
 					(unit 1)
 				)
@@
 		(on_board yes)
 		(dnp no)
-		(property "Reference" "C15"
+		(property "Reference" "C17"
 			(at 114.046 50.038 90)
 			(effects
@@
 			(project ""
 				(path "/27f0531a-0a2b-4c68-af50-4332bf165b5a/f7d1483b-b2e1-4d1b-a579-3453a4da28ca"
-					(reference "C15")
+					(reference "C17")
 					(unit 1)
 				)
@@
 		(on_board yes)
 		(dnp no)
-		(property "Reference" "#PWR018"
+		(property "Reference" "#PWR027"
 			(at 101.6 69.85 0)
 			(effects
@@
 			(project "P1012202501-Cover Sheet"
 				(path "/27f0531a-0a2b-4c68-af50-4332bf165b5a/f7d1483b-b2e1-4d1b-a579-3453a4da28ca"
-					(reference "#PWR018")
+					(reference "#PWR027")
 					(unit 1)
 				)

Commit message: Added new content from the stream.
Parts:
- removed TP8, TP9: TP5010, CONNECTORS:5010, symbol CONNECTORS:TP5010

Commit message: Added new content from latest stream.
Parts:
- removed IC4: USP485REN-L_TR, COMPONENTS:SOIC-8, symbol COMPONENTS:USP485REN-L_TR
- added IC4: USP3485CN-L/TR, COMPONENTS:SOIC-8, symbol COMPONENTS:USP3485CN-L/TR
Connections:
- net 485_DIR: now also IC4.2 (~{RE}), IC4.3 (DE)
- net 485_RX: now also IC4.1 (RO)
- net 485_TX: now also IC4.4 (DI)
- net GND: now also IC4.5 (GND)
- net at CN2.1, D4.2, R5.1: now also IC4.7 (B)
- net at CN2.2, D4.1, J1.2: now also IC4.6 (A)
- net +5V renamed +3V3
- net +3V3: now also IC4.8 (VCC)

Commit message: Added new content from stream.
Other:
- note added: "2"
Changed lines of the file:
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@@
 	(generator_version "9.0")
 	(paper "A4")
+	(text "2"
+		(exclude_from_sim no)
+		(at 268.986 193.548 0)
+		(effects
+			(font
+				(size 1.27 1.27)
+			)
+		)
+	)
 	(text "RS-485"
 		(exclude_from_sim yes)
