File: _Projects/P1012202501-ESP32_Stepper_Controller/Hardware/P1012202501-ESP32_Stepper_Controller/P1012202501-USB UART.kicad_sch (KiCad schematic)
At the start: 8 parts, among them IC5 UCP2102C-A01-GQFN28

Commit message: Added new content from stream.
Parts:
- added CN5: KUSB4105-GF-A, CONNECTORS:GCT_USB4105-GF-A, symbol CONNECTORS:KUSB4105-GF-A
- added D5, D6: TVSCDSOT23-SM712, COMPONENTS:SOT-23-3, symbol COMPONENTS:TVSCDSOT23-SM712
- added Q7: QBC847BDW1T1G, COMPONENTS:SC-70-6, symbol COMPONENTS:QBC847BDW1T1G
- added R21, R22: RC060310K2075AAA, COMPONENTS:RES-0603, symbol COMPONENTS:RC060310K2075AAA
- added S1, S2: SW435151014845, COMPONENTS:435151014845, symbol COMPONENTS:SW435151014845
- added TP18, TP19, TP20, TP21, TP22, TP23, TP24, TP25: TP5010, CONNECTORS:5010, symbol CONNECTORS:TP5010
Connections:
- net DTR: now also Q7.1 (E2), R21.1, TP23.1
- net GND: now also CN5.A1_B12 (GND), CN5.B1_A12 (GND__1), CN5.SH1 (SHELL_GND), CN5.SH2 (SHELL_GND__1), CN5.SH3 (SHELL_GND__2), CN5.SH4 (SHELL_GND__3), D5.3, D6.3, S1.1 (NO_1), S1.2 (NO_2), S1.5 (GND_1), S1.6 (GND_2), S2.1 (NO_1), S2.2 (NO_2), S2.5 (GND_1), S2.6 (GND_2), TP21.1
- net RTS: now also Q7.4 (E1), R22.2, TP22.1
- net USB_D_N: now also CN5.A7 (DN1), CN5.B7 (DN2), D5.2, TP19.1
- net USB_D_P: now also CN5.A6 (DP1), CN5.B6 (DP2), D5.1, TP18.1
- net VBUS: now also CN5.A4_B9 (VBUS), CN5.B4_A9 (VBUS__1), D6.1, TP20.1
- new net: Q7.2 (B2), R22.1
- new net: Q7.5 (B1), R21.2
- new net BOOT_MODE: Q7.6 (C2), S1.3 (COM_1), S1.4 (COM_2), TP24.1
- new net ESP_EN: Q7.3 (C1), S2.3 (COM_1), S2.4 (COM_2), TP25.1
- no-connect marks 6 -> 11
Other:
- moved on the sheet: C18, C19, C20, C21, IC5, R18, R19, R20

Commit message: Added new items from stream.
Parts:
- renumbered C20 to C18, C21 to C19, C18 to C20, C19 to C21, R19 to R18, R20 to R19, R22 to R20, R18 to R22, TP22 to TP18, TP23 to TP19, TP24 to TP20, TP25 to TP21, TP18 to TP22, TP19 to TP23, TP20 to TP24, TP21 to TP25
Changed lines of the file:
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@@
 		(on_board yes)
 		(dnp no)
-		(property "Reference" "R22"
+		(property "Reference" "R20"
 			(at 54.102 142.24 0)
 			(effects
@@
 			(project ""
 				(path "/27f0531a-0a2b-4c68-af50-4332bf165b5a/feaad8cd-dddc-40a5-8f74-4d288b5af2d8"
-					(reference "R22")
+					(reference "R20")
 					(unit 1)
 				)
@@
 		(dnp no)
 		(fields_autoplaced yes)
-		(property "Reference" "#PWR053"
+		(property "Reference" "#PWR049"
 			(at 59.69 97.79 0)
 			(effects
@@
 			(project "P1012202501-Cover Sheet"
 				(path "/27f0531a-0a2b-4c68-af50-4332bf165b5a/feaad8cd-dddc-40a5-8f74-4d288b5af2d8"
-					(reference "#PWR053")
+					(reference "#PWR049")
 					(unit 1)
 				)
@@
 		(dnp no)
 		(fields_autoplaced yes)
-		(property "Reference" "TP24"
+		(property "Reference" "TP20"
 			(at 182.88 124.4599 0)
 			(effects
@@
 			(project ""
 				(path "/27f0531a-0a2b-4c68-af50-4332bf165b5a/feaad8cd-dddc-40a5-8f74-4d288b5af2d8"
-					(reference "TP24")
+					(reference "TP20")
 					(unit 1)
 				)
@@
 		(on_board yes)
 		(dnp no)
-		(property "Reference" "C19"
+		(property "Reference" "C21"
 			(at 130.81 29.2099 90)
 			(effects
@@
 			(project ""
 				(path "/27f0531a-0a2b-4c68-af50-4332bf165b5a/feaad8cd-dddc-40a5-8f74-4d288b5af2d8"
-					(reference "C19")
+					(reference "C21")
 					(unit 1)
 				)
@@
 		(on_board yes)
 		(dnp no)
-		(property "Reference" "C21"
+		(property "Reference" "C19"
 			(at 77.47 74.9299 90)
 			(effects
@@
 			(project ""
 				(path "/27f0531a-0a2b-4c68-af50-4332bf165b5a/feaad8cd-dddc-40a5-8f74-4d288b5af2d8"
-					(reference "C21")
+					(reference "C19")
 					(unit 1)
 				)
@@
 		(dnp no)
 		(fields_autoplaced yes)
-		(property "Reference" "#PWR055"
+		(property "Reference" "#PWR059"
 			(at 273.05 73.66 0)
 			(effects
@@
 			(project "P1012202501-Cover Sheet"
 				(path "/27f0531a-0a2b-4c68-af50-4332bf165b5a/feaad8cd-dddc-40a5-8f74-4d288b5af2d8"
-					(reference "#PWR055")
+					(reference "#PWR059")
 					(unit 1)
 				)
@@
 		(dnp no)
 		(fields_autoplaced yes)
-		(property "Reference" "#PWR060"
+		(property "Reference" "#PWR061"
 			(at 280.67 163.83 0)
 			(effects
@@
 			(project "P1012202501-Cover Sheet"
 				(path "/27f0531a-0a2b-4c68-af50-4332bf165b5a/feaad8cd-dddc-40a5-8f74-4d288b5af2d8"
-					(reference "#PWR060")
+					(reference "#PWR061")
 					(unit 1)
 				)
@@
 		(dnp no)
 		(fields_autoplaced yes)
-		(property "Reference" "#PWR058"
+		(property "Reference" "#PWR052"
 			(at 135.89 135.89 0)
 			(effects
@@
 			(project "P1012202501-Cover Sheet"
 				(path "/27f0531a-0a2b-4c68-af50-4332bf165b5a/feaad8cd-dddc-40a5-8f74-4d288b5af2d8"
-					(reference "#PWR058")
+					(reference "#PWR052")
 					(unit 1)
 				)
@@
 		(on_board yes)
 		(dnp no)
-		(property "Reference" "#PWR057"
+		(property "Reference" "#PWR056"
 			(at 232.41 101.6 0)
 			(effects
@@
 			(project "P1012202501-Cover Sheet"
 				(path "/27f0531a-0a2b-4c68-af50-4332bf165b5a/feaad8cd-dddc-40a5-8f74-4d288b5af2d8"
-					(reference "#PWR057")
+					(reference "#PWR056")
 					(unit 1)
 				)
@@
 		(dnp no)
 		(fields_autoplaced yes)
-		(property "Reference" "#PWR048"
+		(property "Reference" "#PWR050"
 			(at 102.87 24.13 0)
 			(effects
@@
 			(project ""
 				(path "/27f0531a-0a2b-4c68-af50-4332bf165b5a/feaad8cd-dddc-40a5-8f74-4d288b5af2d8"
-					(reference "#PWR048")
+					(reference "#PWR050")
 					(unit 1)
 				)
@@
 		(dnp no)
 		(fields_autoplaced yes)
-		(property "Reference" "TP21"
+		(property "Reference" "TP25"
 			(at 267.97 147.32 0)
 			(effects
@@
 			(project ""
 				(path "/27f0531a-0a2b-4c68-af50-4332bf165b5a/feaad8cd-dddc-40a5-8f74-4d288b5af2d8"
-					(reference "TP21")
+					(reference "TP25")
 					(unit 1)
 				)
@@
 		(dnp no)
 		(fields_autoplaced yes)
-		(property "Reference" "R18"
+		(property "Reference" "R22"
 			(at 175.26 41.9099 90)
 			(effects
@@
 			(project ""
 				(path "/27f0531a-0a2b-4c68-af50-4332bf165b5a/feaad8cd-dddc-40a5-8f74-4d288b5af2d8"
-					(reference "R18")
+					(reference "R22")
 					(unit 1)
 				)
@@
 		(dnp no)
 		(fields_autoplaced yes)
-		(property "Reference" "TP25"
+		(property "Reference" "TP21"
 			(at 182.88 156.2099 0)
 			(effects
@@
 			(project ""
 				(path "/27f0531a-0a2b-4c68-af50-4332bf165b5a/feaad8cd-dddc-40a5-8f74-4d288b5af2d8"
-					(reference "TP25")
+					(reference "TP21")
 					(unit 1)
 				)
@@
 		(on_board yes)
 		(dnp no)
-		(property "Reference" "#PWR054"
+		(property "Reference" "#PWR058"
 			(at 273.05 30.48 0)
 			(effects
@@
 			(project "P1012202501-Cover Sheet"
 				(path "/27f0531a-0a2b-4c68-af50-4332bf165b5a/feaad8cd-dddc-40a5-8f74-4d288b5af2d8"
-					(reference "#PWR054")
+					(reference "#PWR058")
 					(unit 1)
 				)
@@
 		(dnp no)
 		(fields_autoplaced yes)
-		(property "Reference" "TP22"
+		(property "Reference" "TP18"
 			(at 46.99 170.18 0)
 			(effects
@@
 			(project ""
 				(path "/27f0531a-0a2b-4c68-af50-4332bf165b5a/feaad8cd-dddc-40a5-8f74-4d288b5af2d8"
-					(reference "TP22")
+					(reference "TP18")
 					(unit 1)
 				)
@@
 		(dnp no)
 		(fields_autoplaced yes)
-		(property "Reference" "#PWR049"
+		(property "Reference" "#PWR054"
 			(at 163.83 101.6 0)
 			(effects
@@
 			(project ""
 				(path "/27f0531a-0a2b-4c68-af50-4332bf165b5a/feaad8cd-dddc-40a5-8f74-4d288b5af2d8"
-					(reference "#PWR049")
+					(reference "#PWR054")
 					(unit 1)
 				)
@@
 		(dnp no)
 		(fields_autoplaced yes)
-		(property "Reference" "TP23"
+		(property "Reference" "TP19"
 			(at 46.99 185.42 0)
 			(effects
@@
 			(project ""
 				(path "/27f0531a-0a2b-4c68-af50-4332bf165b5a/feaad8cd-dddc-40a5-8f74-4d288b5af2d8"
-					(reference "TP23")
+					(reference "TP19")
 					(unit 1)
 				)
@@
 		(on_board yes)
 		(dnp no)
-		(property "Reference" "#PWR052"
+		(property "Reference" "#PWR048"
 			(at 17.78 62.23 0)
 			(effects
@@
 			(project ""
 				(path "/27f0531a-0a2b-4c68-af50-4332bf165b5a/feaad8cd-dddc-40a5-8f74-4d288b5af2d8"
-					(reference "#PWR052")
+					(reference "#PWR048")
 					(unit 1)
 				)
@@
 		(dnp no)
 		(fields_autoplaced yes)
-		(property "Reference" "#PWR059"
+		(property "Reference" "#PWR053"
 			(at 135.89 167.64 0)
 			(effects
@@
 			(project "P1012202501-Cover Sheet"
 				(path "/27f0531a-0a2b-4c68-af50-4332bf165b5a/feaad8cd-dddc-40a5-8f74-4d288b5af2d8"
-					(reference "#PWR059")
+					(reference "#PWR053")
 					(unit 1)
 				)
@@
 		(dnp no)
 		(fields_autoplaced yes)
-		(property "Reference" "R19"
+		(property "Reference" "R18"
 			(at 30.48 58.42 0)
 			(effects
@@
 			(project ""
 				(path "/27f0531a-0a2b-4c68-af50-4332bf165b5a/feaad8cd-dddc-40a5-8f74-4d288b5af2d8"
-					(reference "R19")
+					(reference "R18")
 					(unit 1)
 				)
@@
 		(dnp no)
 		(fields_autoplaced yes)
-		(property "Reference" "TP18"
+		(property "Reference" "TP22"
 			(at 193.04 19.05 0)
 			(effects
@@
 			(project ""
 				(path "/27f0531a-0a2b-4c68-af50-4332bf165b5a/feaad8cd-dddc-40a5-8f74-4d288b5af2d8"
-					(reference "TP18")
+					(reference "TP22")
 					(unit 1)
 				)
@@
 		(dnp no)
 		(fields_autoplaced yes)
-		(property "Reference" "TP20"
+		(property "Reference" "TP24"
 			(at 267.97 134.62 0)
 			(effects
@@
 			(project ""
 				(path "/27f0531a-0a2b-4c68-af50-4332bf165b5a/feaad8cd-dddc-40a5-8f74-4d288b5af2d8"
-					(reference "TP20")
+					(reference "TP24")
 					(unit 1)
 				)
@@
 		(dnp no)
 		(fields_autoplaced yes)
-		(property "Reference" "#PWR050"
+		(property "Reference" "#PWR055"
 			(at 172.72 34.29 0)
 			(effects
@@
 			(project "P1012202501-Cover Sheet"
 				(path "/27f0531a-0a2b-4c68-af50-4332bf165b5a/feaad8cd-dddc-40a5-8f74-4d288b5af2d8"
-					(reference "#PWR050")
+					(reference "#PWR055")
 					(unit 1)
 				)
@@
 		(dnp no)
 		(fields_autoplaced yes)
-		(property "Reference" "#PWR056"
+		(property "Reference" "#PWR057"
 			(at 264.16 113.03 0)
 			(effects
@@
 			(project "P1012202501-Cover Sheet"
 				(path "/27f0531a-0a2b-4c68-af50-4332bf165b5a/feaad8cd-dddc-40a5-8f74-4d288b5af2d8"
-					(reference "#PWR056")
+					(reference "#PWR057")
 					(unit 1)
 				)
@@
 		(on_board yes)
 		(dnp no)
-		(property "Reference" "C18"
+		(property "Reference" "C20"
 			(at 115.57 29.2099 90)
 			(effects
@@
 			(project ""
 				(path "/27f0531a-0a2b-4c68-af50-4332bf165b5a/feaad8cd-dddc-40a5-8f74-4d288b5af2d8"
-					(reference "C18")
+					(reference "C20")
 					(unit 1)
 				)
@@
 		(on_board yes)
 		(dnp no)
-		(property "Reference" "C20"
+		(property "Reference" "C18"
 			(at 63.5 74.9299 90)
 			(effects
@@
 			(project ""
 				(path "/27f0531a-0a2b-4c68-af50-4332bf165b5a/feaad8cd-dddc-40a5-8f74-4d288b5af2d8"
-					(reference "C20")
+					(reference "C18")
 					(unit 1)
 				)
@@
 		(dnp no)
 		(fields_autoplaced yes)
-		(property "Reference" "R20"
+		(property "Reference" "R19"
 			(at 45.72 77.4699 90)
 			(effects
@@
 			(project ""
 				(path "/27f0531a-0a2b-4c68-af50-4332bf165b5a/feaad8cd-dddc-40a5-8f74-4d288b5af2d8"
-					(reference "R20")
+					(reference "R19")
 					(unit 1)
 				)
@@
 		(dnp no)
 		(fields_autoplaced yes)
-		(property "Reference" "TP19"
+		(property "Reference" "TP23"
 			(at 193.04 35.56 0)
 			(effects
@@
 			(project ""
 				(path "/27f0531a-0a2b-4c68-af50-4332bf165b5a/feaad8cd-dddc-40a5-8f74-4d288b5af2d8"
-					(reference "TP19")
+					(reference "TP23")
 					(unit 1)
 				)
@@
 		(on_board yes)
 		(dnp no)
-		(property "Reference" "#PWR061"
+		(property "Reference" "#PWR060"
 			(at 280.67 142.24 0)
 			(effects
@@
 			(project "P1012202501-Cover Sheet"
 				(path "/27f0531a-0a2b-4c68-af50-4332bf165b5a/feaad8cd-dddc-40a5-8f74-4d288b5af2d8"
-					(reference "#PWR061")
+					(reference "#PWR060")
 					(unit 1)
 				)

Commit message: Added items from latest stream.
Parts:
- added D7: TVSCDSOT23-SM712, COMPONENTS:SOT-23-3, symbol COMPONENTS:TVSCDSOT23-SM712
Connections:
- net BOOT_MODE: now also D7.1
- net ESP_EN: now also D7.2
- net GND: now also D7.3
- net +3.3V renamed +3V3

Commit message: Added new content from stream.
Parts:
- IC5: symbol COMPONENTS:UCP2102C-A01-GQFN28 -> COMPONENTS:UCP2102N-A02-GQFN28R; Manufacturer 1 P/N CP2102C-A01-GQFN28 -> CP2102N-A02-GQFN28R; Vendor 1a Cost HV 1.31 -> 2.13; Vendor 1a Cost LV 3.55 -> 3.52; Vendor 1a P/N 634-P2102CA01GQFN28 -> 634-CP2102NA02QFN28R
Connections:
- no-connect marks 11 -> 21
Other:
- note added: "2"
Changed lines of the file:
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@@
 	(generator_version "9.0")
 	(paper "A4")
+	(text "2"
+		(exclude_from_sim no)
+		(at 268.986 193.294 0)
+		(effects
+			(font
+				(size 1.27 1.27)
+			)
+		)
+	)
 	(text "USB UART"
 		(exclude_from_sim yes)
@@
 	)
 	(no_connect
+		(at 160.02 64.77)
+	)
+	(no_connect
 		(at 228.6 62.23)
 	)
@@
 	)
 	(no_connect
+		(at 160.02 82.55)
+	)
+	(no_connect
+		(at 160.02 74.93)
+	)
+	(no_connect
+		(at 160.02 77.47)
+	)
+	(no_connect
+		(at 160.02 85.09)
+	)
+	(no_connect
 		(at 116.84 82.55)
 	)
 	(no_connect
+		(at 160.02 67.31)
+	)
+	(no_connect
 		(at 116.84 87.63)
 	)
 	(no_connect
+		(at 160.02 72.39)
+	)
+	(no_connect
 		(at 116.84 90.17)
 	)
 	(no_connect
+		(at 160.02 87.63)
+	)
+	(no_connect
 		(at 116.84 72.39)
 	)
 	(no_connect
+		(at 160.02 69.85)
+	)
+	(no_connect
 		(at 116.84 92.71)
 	)
@@
 		(at 228.6 57.15)
 	)
+	(no_connect
+		(at 160.02 80.01)
+	)
 	(wire
 		(pts
@@
 	)
 	(symbol
-		(lib_id "COMPONENTS:UCP2102C-A01-GQFN28")
+		(lib_id "COMPONENTS:UCP2102N-A02-GQFN28R")
 		(at 116.84 52.07 0)
 		(unit 1)
@@
 			)
 		)
-		(property "Description" "Interface IC, USB to UART Bridge, QFN28, -40°C to +85°C, RoHS"
+		(property "Description" "Interface IC, USB to UART Bridge, USB 2.0, Full Speed, QFN28, -40°C to +85°C, RoHS"
 			(at 85.344 33.274 0)
 			(effects
@@
 			)
 		)
-		(property "Manufacturer 1 P/N" "CP2102C-A01-GQFN28"
+		(property "Manufacturer 1 P/N" "CP2102N-A02-GQFN28R"
 			(at 82.296 28.448 0)
 			(effects
@@
 			)
 		)
-		(property "Vendor 1a P/N" "634-P2102CA01GQFN28"
+		(property "Vendor 1a P/N" "634-CP2102NA02QFN28R"
 			(at 82.55 36.068 0)
 			(effects
@@
 			)
 		)
-		(property "Vendor 1a Cost LV" "3.55"
+		(property "Vendor 1a Cost LV" "3.52"
 			(at 100.33 21.336 0)
 			(effects
@@
 			)
 		)
-		(property "Vendor 1a Cost HV" "1.31"
+		(property "Vendor 1a Cost HV" "2.13"
 			(at 93.218 12.446 0)
 			(effects
