File: _Projects/P1012202501-ESP32_Stepper_Controller/Hardware/P1012202501-ESP32_Stepper_Controller/P1012202501-Stepper Driver.kicad_sch (KiCad schematic)
At the start: 1 part, among them CN6 KPTBP04R1-500-04BE

Commit message: Added new content from recent stream.
Parts:
- added C22, C23, C24: CC0603104050AAAX7R, COMPONENTS:CAP-0603, symbol COMPONENTS:CC0603104050AAAX7R
- added C25: CEA771MS107M1JLAS018, COMPONENTS:A768MS157M1HLAE024, symbol COMPONENTS:CEA771MS107M1JLAS018
- added C26: CC0603103050AAAX7R, COMPONENTS:CAP-0603, symbol COMPONENTS:CC0603103050AAAX7R
- added IC6: UDRV8825PWPR, COMPONENTS:HTSSOP-28, symbol COMPONENTS:UDRV8825PWPR
- added R23: RC06031M0075AAA, COMPONENTS:RES-0603, symbol COMPONENTS:RC06031M0075AAA
- added R24, R25: RC08050R2075AAE, COMPONENTS:RES-0805, symbol COMPONENTS:RC08050R2075AAE
Connections:
- net +24V: now also C22.1, C23.1, C24.1, C25.1 (+), IC6.11 (VMB), IC6.4 (VMA), R23.1
- net GND: now also C22.2, C23.2, C25.2 (-), IC6.14 (GND_1), IC6.28 (GND_2), IC6.29 (GND_3), R24.2, R25.2
- new net: IC6.9 (ISENB), R25.1
- new net: C26.1, IC6.1 (CP1)
- new net: C26.2, IC6.2 (CP2)
- new net: IC6.6 (ISENA), R24.1
- new net: C24.2, IC6.3 (VCP), R23.2
Other:
- moved on the sheet: CN6

Commit message: Adding new materials from stream.
Parts:
- added C27: CC0603474050AAAX7R, COMPONENTS:CAP-0603, symbol COMPONENTS:CC0603474050AAAX7R
- added CN7: KHS4B-PH-SM4-TB(LF)(SN), CONNECTORS:S4B-PH-SM4-TB, symbol CONNECTORS:KHS4B-PH-SM4-TB(LF)(SN)
- added R26: RC060350K075AAA, COMPONENTS:RES-0603, symbol COMPONENTS:RC060350K075AAA
- added R27: RC060330K075AAA, COMPONENTS:RES-0603, symbol COMPONENTS:RC060330K075AAA
- added R28, R29, R30: RC060310K2075AAA, COMPONENTS:RES-0603, symbol COMPONENTS:RC060310K2075AAA
Connections:
- net GND: now also C27.2, CN7.4, R27.2
- net at CN6.1: now also IC6.10 (BOUT1)
- net at CN6.2: now also IC6.8 (BOUT2)
- net at CN6.3: now also IC6.7 (AOUT2)
- net at CN6.4: now also IC6.5 (AOUT1)
- net at IC6.12 (AVREF): now also IC6.13 (BVREF), R26.2, R27.1
- net at IC6.15 (V3P3OUT): now also C27.1, R26.1
- net STP_RESET: now reaches IC6.16 (NRESET)
- net STP_RESET: now also R30.2
- net +3V3: now reaches IC6.17 (NSLEEP)
- net +3V3: now also R28.1, R29.1, R30.1
- net STP_FLT: now reaches IC6.18 (NFAULT)
- net STP_FLT: now also R28.2
- net STP_DIR: now reaches IC6.20 (DIR)
- net STP_ENABLE: now reaches IC6.21 (NENBL)
- net STP_ENABLE: now also R29.2
- net STP_STEP: now reaches IC6.22 (STEP)
- net STP_MS0: now reaches IC6.24 (MODE0)
- net STP_MS1: now reaches IC6.25 (MODE1)
- net STP_MS2: now reaches IC6.26 (MODE2)
- new net +5V: CN7.1
- new net FAN_PWM: CN7.3
- new net FAN_TACH: CN7.2
- no-connect marks 0 -> 2
Other:
- moved on the sheet: CN6

Commit message: Added new items from stream.
Parts:
- renumbered C25 to C22, C22 to C23, C23 to C24, C24 to C25, CN7 to CN6, CN6 to CN7, R29 to R23, R30 to R24, R23 to R25, R24 to R26, R25 to R27, R26 to R28, R27 to R29, R28 to R30
Changed lines of the file:
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@@
 		(dnp no)
 		(fields_autoplaced yes)
-		(property "Reference" "#PWR070"
+		(property "Reference" "#PWR062"
 			(at 24.13 125.73 0)
 			(effects
@@
 			(project "P1012202501-Cover Sheet"
 				(path "/27f0531a-0a2b-4c68-af50-4332bf165b5a/2932f4ee-8c5b-459c-9bd5-5a172fd29c3b"
-					(reference "#PWR070")
+					(reference "#PWR062")
 					(unit 1)
 				)
@@
 		(dnp no)
 		(fields_autoplaced yes)
-		(property "Reference" "#PWR072"
+		(property "Reference" "#PWR065"
 			(at 67.31 170.18 0)
 			(effects
@@
 			(project "P1012202501-Cover Sheet"
 				(path "/27f0531a-0a2b-4c68-af50-4332bf165b5a/2932f4ee-8c5b-459c-9bd5-5a172fd29c3b"
-					(reference "#PWR072")
+					(reference "#PWR065")
 					(unit 1)
 				)
@@
 		(dnp no)
 		(fields_autoplaced yes)
-		(property "Reference" "R27"
+		(property "Reference" "R29"
 			(at 193.04 137.1599 90)
 			(effects
@@
 			(project ""
 				(path "/27f0531a-0a2b-4c68-af50-4332bf165b5a/2932f4ee-8c5b-459c-9bd5-5a172fd29c3b"
-					(reference "R27")
+					(reference "R29")
 					(unit 1)
 				)
@@
 		(dnp no)
 		(fields_autoplaced yes)
-		(property "Reference" "#PWR066"
+		(property "Reference" "#PWR071"
 			(at 208.28 127 0)
 			(effects
@@
 			(project "P1012202501-Cover Sheet"
 				(path "/27f0531a-0a2b-4c68-af50-4332bf165b5a/2932f4ee-8c5b-459c-9bd5-5a172fd29c3b"
-					(reference "#PWR066")
+					(reference "#PWR071")
 					(unit 1)
 				)
@@
 		(on_board yes)
 		(dnp no)
-		(property "Reference" "CN6"
+		(property "Reference" "CN7"
 			(at 194.31 90.1701 0)
 			(effects
@@
 			(project ""
 				(path "/27f0531a-0a2b-4c68-af50-4332bf165b5a/2932f4ee-8c5b-459c-9bd5-5a172fd29c3b"
-					(reference "CN6")
+					(reference "CN7")
 					(unit 1)
 				)
@@
 		(dnp no)
 		(fields_autoplaced yes)
-		(property "Reference" "#PWR069"
+		(property "Reference" "#PWR068"
 			(at 132.08 83.82 0)
 			(effects
@@
 			(project "P1012202501-Cover Sheet"
 				(path "/27f0531a-0a2b-4c68-af50-4332bf165b5a/2932f4ee-8c5b-459c-9bd5-5a172fd29c3b"
-					(reference "#PWR069")
+					(reference "#PWR068")
 					(unit 1)
 				)
@@
 		(dnp no)
 		(fields_autoplaced yes)
-		(property "Reference" "R26"
+		(property "Reference" "R28"
 			(at 193.04 114.2999 90)
 			(effects
@@
 			(project ""
 				(path "/27f0531a-0a2b-4c68-af50-4332bf165b5a/2932f4ee-8c5b-459c-9bd5-5a172fd29c3b"
-					(reference "R26")
+					(reference "R28")
 					(unit 1)
 				)
@@
 		(dnp no)
 		(fields_autoplaced yes)
-		(property "Reference" "R25"
+		(property "Reference" "R27"
 			(at 132.08 123.1899 90)
 			(effects
@@
 			(project ""
 				(path "/27f0531a-0a2b-4c68-af50-4332bf165b5a/2932f4ee-8c5b-459c-9bd5-5a172fd29c3b"
-					(reference "R25")
+					(reference "R27")
 					(unit 1)
 				)
@@
 		(on_board yes)
 		(dnp no)
-		(property "Reference" "C25"
+		(property "Reference" "C22"
 			(at 29.21 80.0099 90)
 			(effects
@@
 			(project ""
 				(path "/27f0531a-0a2b-4c68-af50-4332bf165b5a/2932f4ee-8c5b-459c-9bd5-5a172fd29c3b"
-					(reference "C25")
+					(reference "C22")
 					(unit 1)
 				)
@@
 		(dnp no)
 		(fields_autoplaced yes)
-		(property "Reference" "R24"
+		(property "Reference" "R26"
 			(at 120.65 123.1899 90)
 			(effects
@@
 			(project ""
 				(path "/27f0531a-0a2b-4c68-af50-4332bf165b5a/2932f4ee-8c5b-459c-9bd5-5a172fd29c3b"
-					(reference "R24")
+					(reference "R26")
 					(unit 1)
 				)
@@
 		(dnp no)
 		(fields_autoplaced yes)
-		(property "Reference" "#PWR062"
+		(property "Reference" "#PWR069"
 			(at 172.72 123.19 0)
 			(effects
@@
 			(project ""
 				(path "/27f0531a-0a2b-4c68-af50-4332bf165b5a/2932f4ee-8c5b-459c-9bd5-5a172fd29c3b"
-					(reference "#PWR062")
+					(reference "#PWR069")
 					(unit 1)
 				)
@@
 		(on_board yes)
 		(dnp no)
-		(property "Reference" "C23"
+		(property "Reference" "C24"
 			(at 59.69 80.0099 90)
 			(effects
@@
 			(project ""
 				(path "/27f0531a-0a2b-4c68-af50-4332bf165b5a/2932f4ee-8c5b-459c-9bd5-5a172fd29c3b"
-					(reference "C23")
+					(reference "C24")
 					(unit 1)
 				)
@@
 		(dnp no)
 		(fields_autoplaced yes)
-		(property "Reference" "R28"
+		(property "Reference" "R30"
 			(at 237.49 83.8199 90)
 			(effects
@@
 			(project ""
 				(path "/27f0531a-0a2b-4c68-af50-4332bf165b5a/2932f4ee-8c5b-459c-9bd5-5a172fd29c3b"
-					(reference "R28")
+					(reference "R30")
 					(unit 1)
 				)
@@
 		(dnp no)
 		(fields_autoplaced yes)
-		(property "Reference" "R29"
+		(property "Reference" "R23"
 			(at 40.64 121.92 0)
 			(effects
@@
 			(project ""
 				(path "/27f0531a-0a2b-4c68-af50-4332bf165b5a/2932f4ee-8c5b-459c-9bd5-5a172fd29c3b"
-					(reference "R29")
+					(reference "R23")
 					(unit 1)
 				)
@@
 		(on_board yes)
 		(dnp no)
-		(property "Reference" "C22"
+		(property "Reference" "C23"
 			(at 44.45 80.0099 90)
 			(effects
@@
 			(project ""
 				(path "/27f0531a-0a2b-4c68-af50-4332bf165b5a/2932f4ee-8c5b-459c-9bd5-5a172fd29c3b"
-					(reference "C22")
+					(reference "C23")
 					(unit 1)
 				)
@@
 		(on_board yes)
 		(dnp no)
-		(property "Reference" "C24"
+		(property "Reference" "C25"
 			(at 76.2 80.0099 90)
 			(effects
@@
 			(project ""
 				(path "/27f0531a-0a2b-4c68-af50-4332bf165b5a/2932f4ee-8c5b-459c-9bd5-5a172fd29c3b"
-					(reference "C24")
+					(reference "C25")
 					(unit 1)
 				)
@@
 		(dnp no)
 		(fields_autoplaced yes)
-		(property "Reference" "#PWR068"
+		(property "Reference" "#PWR072"
 			(at 234.95 76.2 0)
 			(effects
@@
 			(project "P1012202501-Cover Sheet"
 				(path "/27f0531a-0a2b-4c68-af50-4332bf165b5a/2932f4ee-8c5b-459c-9bd5-5a172fd29c3b"
-					(reference "#PWR068")
+					(reference "#PWR072")
 					(unit 1)
 				)
@@
 		(dnp no)
 		(fields_autoplaced yes)
-		(property "Reference" "#PWR067"
+		(property "Reference" "#PWR070"
 			(at 190.5 158.75 0)
 			(effects
@@
 			(project "P1012202501-Cover Sheet"
 				(path "/27f0531a-0a2b-4c68-af50-4332bf165b5a/2932f4ee-8c5b-459c-9bd5-5a172fd29c3b"
-					(reference "#PWR067")
+					(reference "#PWR070")
 					(unit 1)
 				)
@@
 		(dnp no)
 		(fields_autoplaced yes)
-		(property "Reference" "#PWR065"
+		(property "Reference" "#PWR067"
 			(at 123.19 143.51 0)
 			(effects
@@
 			(project "P1012202501-Cover Sheet"
 				(path "/27f0531a-0a2b-4c68-af50-4332bf165b5a/2932f4ee-8c5b-459c-9bd5-5a172fd29c3b"
-					(reference "#PWR065")
+					(reference "#PWR067")
 					(unit 1)
 				)
@@
 		(on_board yes)
 		(dnp no)
-		(property "Reference" "CN7"
+		(property "Reference" "CN6"
 			(at 42.926 161.544 0)
 			(effects
@@
 			(project ""
 				(path "/27f0531a-0a2b-4c68-af50-4332bf165b5a/2932f4ee-8c5b-459c-9bd5-5a172fd29c3b"
-					(reference "CN7")
+					(reference "CN6")
 					(unit 1)
 				)
@@
 		(dnp no)
 		(fields_autoplaced yes)
-		(property "Reference" "R30"
+		(property "Reference" "R24"
 			(at 40.64 133.35 0)
 			(effects
@@
 			(project ""
 				(path "/27f0531a-0a2b-4c68-af50-4332bf165b5a/2932f4ee-8c5b-459c-9bd5-5a172fd29c3b"
-					(reference "R30")
+					(reference "R24")
 					(unit 1)
 				)
@@
 		(on_board yes)
 		(dnp no)
-		(property "Reference" "R23"
+		(property "Reference" "R25"
 			(at 86.614 80.264 90)
 			(effects
@@
 			(project ""
 				(path "/27f0531a-0a2b-4c68-af50-4332bf165b5a/2932f4ee-8c5b-459c-9bd5-5a172fd29c3b"
-					(reference "R23")
+					(reference "R25")
 					(unit 1)
 				)
@@
 		(dnp no)
 		(fields_autoplaced yes)
-		(property "Reference" "#PWR071"
+		(property "Reference" "#PWR066"
 			(at 67.31 185.42 0)
 			(effects
@@
 			(project "P1012202501-Cover Sheet"
 				(path "/27f0531a-0a2b-4c68-af50-4332bf165b5a/2932f4ee-8c5b-459c-9bd5-5a172fd29c3b"
-					(reference "#PWR071")
+					(reference "#PWR066")
 					(unit 1)
 				)

Commit message: Added new content and changes from stream.
Connections:
- net at CN7.1: now also IC6.5 (AOUT1); no longer IC6.10 (BOUT1)
- net at CN7.2: now also IC6.7 (AOUT2); no longer IC6.8 (BOUT2)
- net at CN7.3: now also IC6.8 (BOUT2); no longer IC6.7 (AOUT2)
- net at CN7.4: now also IC6.10 (BOUT1); no longer IC6.5 (AOUT1)

Commit message: Added items from latest stream.
Parts:
- added R31: RC06031K0075AAA, COMPONENTS:RES-0603, symbol COMPONENTS:RC06031K0075AAA
Connections:
- net +3V3: now also R31.1
- net FAN_TACH: now also R31.2
Changed lines of the file:
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@@
 	)
 	(junction
+		(at 80.01 171.45)
+		(diameter 0)
+		(color 0 0 0 0)
+	)
+	(junction
 		(at 72.39 69.85)
 		(diameter 0)
@@
 	(wire
 		(pts
+			(xy 80.01 146.05) (xy 80.01 149.86)
+		)
+		(stroke
+			(width 0)
+			(type default)
+		)
+	)
+	(wire
+		(pts
 			(xy 170.18 113.03) (xy 172.72 113.03)
 		)
@@
 	(wire
 		(pts
+			(xy 80.01 171.45) (xy 87.63 171.45)
+		)
+		(stroke
+			(width 0)
+			(type default)
+		)
+	)
+	(wire
+		(pts
 			(xy 105.41 106.68) (xy 105.41 153.67)
 		)
@@
 	(wire
 		(pts
-			(xy 57.15 171.45) (xy 67.31 171.45)
+			(xy 57.15 171.45) (xy 80.01 171.45)
 		)
 		(stroke
@@
 	(wire
 		(pts
+			(xy 80.01 167.64) (xy 80.01 171.45)
+		)
+		(stroke
+			(width 0)
+			(type default)
+		)
+	)
+	(wire
+		(pts
 			(xy 234.95 72.39) (xy 234.95 76.2)
 		)
@@
 	(global_label "FAN_TACH"
 		(shape output)
-		(at 67.31 171.45 0)
+		(at 87.63 171.45 0)
 		(fields_autoplaced yes)
 		(effects
@@
 		)
 		(property "Intersheetrefs" "${INTERSHEET_REFS}"
-			(at 79.4272 171.45 0)
+			(at 99.7472 171.45 0)
 			(effects
 				(font
@@
 	)
 	(symbol
+		(lib_id "COMPONENTS:RC06031K0075AAA")
+		(at 80.01 149.86 270)
+		(unit 1)
+		(exclude_from_sim no)
+		(in_bom yes)
+		(on_board yes)
+		(dnp no)
+		(fields_autoplaced yes)
+		(property "Reference" "R31"
+			(at 82.55 157.4799 90)
+			(effects
+				(font
+					(size 1.27 1.27)
+				)
+				(justify left)
+			)
+		)
+		(property "Value" "RC06031K0075AAA"
+			(at 73.914 151.384 0)
+			(effects
+				(font
+					(size 1.27 1.27)
+				)
+				(justify left top)
+				(hide yes)
+			)
+		)
+		(property "Footprint" "COMPONENTS:RES-0603"
+			(at -16.18 163.83 0)
+			(effects
+				(font
+					(size 1.27 1.27)
+				)
+				(justify left top)
+				(hide yes)
+			)
+		)
+		(property "Datasheet" ""
+			(at -116.18 163.83 0)
+			(effects
+				(font
+					(size 1.27 1.27)
+				)
+				(justify left top)
+				(hide yes)
+			)
+		)
+		(property "Description" "Resistor, Chip, 0603, 1KΩ, 75V, 5%, -55°C to 155°C, RoHS, AEC-Q200"
+			(at 70.866 153.924 0)
+			(effects
+				(font
+					(size 1.27 1.27)
+				)
+				(hide yes)
+			)
+		)
+		(property "Manufacturer 1" "Yageo"
+			(at 64.516 147.32 0)
+			(effects
+				(font
+					(size 1.27 1.27)
+				)
+				(hide yes)
+			)
+		)
+		(property "Manufacturer 1 P/N" "SR0603JR-071KL"
+			(at 66.802 156.972 0)
+			(effects
+				(font
+					(size 1.27 1.27)
+				)
+				(hide yes)
+			)
+		)
+		(property "Vendor 1a" "Mouser"
+			(at 82.296 130.048 0)
+			(effects
+				(font
+					(size 1.27 1.27)
+				)
+				(hide yes)
+			)
+		)
+		(property "Vendor 1a P/N" "603-SR0603JR-071KL"
+			(at 90.424 146.05 0)
+			(effects
+				(font
+					(size 1.27 1.27)
+				)
+				(hide yes)
+			)
+		)
+		(property "Vendor 1a Cost LV" "0.11"
+			(at 79.756 131.064 0)
+			(effects
+				(font
+					(size 1.27 1.27)
+				)
+				(hide yes)
+			)
+		)
+		(property "Vendor 1a Cost HV" "0.031"
+			(at 86.36 131.572 0)
+			(effects
+				(font
+					(size 1.27 1.27)
+				)
+				(hide yes)
+			)
+		)
+		(property "Val" "1KΩ"
+			(at 82.55 160.0199 90)
+			(effects
+				(font
+					(size 1.27 1.27)
+				)
+				(justify left)
+			)
+		)
+		(pin "1"
+		)
+		(pin "2"
+		)
+		(instances
+			(project ""
+				(path "/27f0531a-0a2b-4c68-af50-4332bf165b5a/2932f4ee-8c5b-459c-9bd5-5a172fd29c3b"
+					(reference "R31")
+					(unit 1)
+				)
+			)
+		)
+	)
+	(symbol
 		(lib_id "COMPONENTS:CC0603104050AAAX7R")
 		(at 55.88 74.93 270)
@@
 					(unit 1)
 				)
+			)
+		)
+	)
+	(symbol
+		(lib_id "power:+3V3")
+		(at 80.01 146.05 0)
+		(unit 1)
+		(exclude_from_sim no)
+		(in_bom yes)
+		(on_board yes)
+		(dnp no)
+		(fields_autoplaced yes)
+		(property "Reference" "#PWR073"
+			(at 80.01 149.86 0)
+			(effects
+				(font
+					(size 1.27 1.27)
+				)
+				(hide yes)
+			)
+		)
+		(property "Value" "+3V3"
+			(at 80.01 140.97 0)
+			(effects
+				(font
+					(size 1.27 1.27)
+				)
+			)
+		)
+		(property "Footprint" ""
+			(at 80.01 146.05 0)
+			(effects
+				(font
+					(size 1.27 1.27)
+				)
+				(hide yes)
+			)
+		)
+		(property "Datasheet" ""
+			(at 80.01 146.05 0)
+			(effects
+				(font
+					(size 1.27 1.27)
+				)
+				(hide yes)
+			)
+		)
+		(property "Description" "Power symbol creates a global label with name \"+3V3\""
+			(at 80.01 146.05 0)
+			(effects
+				(font
+					(size 1.27 1.27)
+				)
+				(hide yes)
+			)
+		)
+		(pin "1"
+		)
+		(instances
+			(project "P1012202501-ESP32_Stepper_Controller"
+				(path "/27f0531a-0a2b-4c68-af50-4332bf165b5a/2932f4ee-8c5b-459c-9bd5-5a172fd29c3b"
+					(reference "#PWR073")
+					(unit 1)
+				)

Commit message: Added latest content from stream.
Parts:
- added C28: CC0603104050AAAX7R, COMPONENTS:CAP-0603, symbol COMPONENTS:CC0603104050AAAX7R
- added C29: CC0603226010AABX5R, COMPONENTS:CAP-0603, symbol COMPONENTS:CC0603226010AABX5R
- added IC7: UTMP36GRTZ-REEL7, COMPONENTS:SOT-23-5, symbol COMPONENTS:UTMP36GRTZ-REEL7
Connections:
- net +3V3: now also C28.1, C29.1, IC7.2 (+VS), IC7.4 (~{SHUTDOWN})
- net GND: now also C28.2, C29.2, IC7.5 (GND)
- new net TEMP_SENSE: IC7.1 (VOUT)

Commit message: Added new content from stream.
Other:
- note added: "2"
Changed lines of the file:
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@@
+		)
+	)
+	(text "2"
+		(exclude_from_sim no)
+		(at 268.986 193.04 0)
+		(effects
+			(font
+				(size 1.27 1.27)
+			)
 		)
 	)

Commit message: Added new items from streams.
Parts:
- added TP26, TP27, TP28, TP29, TP30, TP31, TP32, TP33, TP34, TP35, TP36: TP5010, CONNECTORS:5010, symbol CONNECTORS:TP5010
Connections:
- net FAN_PWM: now also TP36.1
- net FAN_TACH: now also TP35.1
- net STP_DIR: now also TP29.1
- net STP_ENABLE: now also TP27.1
- net STP_FLT: now also TP34.1
- net STP_MS0: now also TP31.1
- net STP_MS1: now also TP32.1
- net STP_MS2: now also TP33.1
- net STP_RESET: now also TP28.1
- net STP_STEP: now also TP30.1
- net TEMP_SENSE: now also TP26.1
Other:
- moved on the sheet: C28, C29, IC7
