File: _Projects/P1012202501-ESP32_Stepper_Controller/Hardware/P1012202501-ESP32_Stepper_Controller/P1012202501-ESP32.kicad_sch (KiCad schematic)
At the start: 6 parts, among them IC3 ESP32-WROOM-32UE-N16

Commit message: Added content from latest stream.
Connections:
- net INPUT_1: now reaches IC3.10 (IO25)
- net INPUT_2: now reaches IC3.11 (IO26)
- net INPUT_3: now reaches IC3.12 (IO27)
- net STP_ENABLE: now reaches IC3.13 (IO14)
- net STP_STEP: now reaches IC3.14 (IO12)
- net STP_RESET: now reaches IC3.16 (IO13)
- net STP_MS0: now reaches IC3.23 (IO15)
- net 485_TX: now reaches IC3.24 (IO2)
- net 485_RX: now reaches IC3.25 (IO0)
- net 485_DIR: now reaches IC3.26 (IO4)
- net STP_MS1: now reaches IC3.27 (IO16)
- net STP_MS2: now reaches IC3.28 (IO17)
- net STP_DIR: now reaches IC3.29 (IO5)
- net STP_FLT: now reaches IC3.30 (IO18)
- net UART_RX: now reaches IC3.31 (IO19)
- net UART_TX: now reaches IC3.33 (IO21)
- net FAN_TACH: now reaches IC3.36 (IO22)
- net FAN_PWM: now reaches IC3.37 (IO23)

Commit message: Adding new content from stream.
Parts:
- added R17: RC060310K2075AAA, COMPONENTS:RES-0603, symbol COMPONENTS:RC060310K2075AAA
Connections:
- net ENABLE is gone; now on net INPUT_3: IC3.6 (IO34)
- net +3V3: now also R17.1
- net 485_DIR: now also IC3.12 (IO27); no longer IC3.26 (IO4)
- net 485_RX: now also IC3.10 (IO25); no longer IC3.25 (IO0)
- net 485_TX: now also IC3.11 (IO26); no longer IC3.24 (IO2)
- net INPUT_1: now also IC3.8 (IO32); no longer IC3.10 (IO25)
- net INPUT_2: now also IC3.9 (IO33); no longer IC3.11 (IO26)
- net INPUT_3: no longer IC3.12 (IO27)
- new net BOOT_MODE: IC3.25 (IO0), R17.2

Commit message: Added new items from stream.
Parts:
- renumbered R1 to R3, R17 to R4
Connections:
- no-connect marks 7 -> 9

Commit message: Added new content from latest stream.
Parts:
- added D8: TVSCDSOT23-SM712, COMPONENTS:SOT-23-3, symbol COMPONENTS:TVSCDSOT23-SM712
- added J4: KH68001-406HLF, CONNECTORS:6x1HDR2.54mm, symbol CONNECTORS:KH68001-406HLF
Connections:
- net GND: now also D8.3, J4.1
- net UART_RX: now also D8.2, J4.4
- net UART_TX: now also D8.1, J4.5
- no-connect marks 9 -> 12

Commit message: Added latest content from stream.
Parts:
- added D9: DLLS R976-NR-1, COMPONENTS:LED-0805, symbol COMPONENTS:DLLS R976-NR-1
- added R32: RC0603330075AAA, COMPONENTS:RES-0603, symbol COMPONENTS:RC0603330075AAA
Connections:
- net GND: now also D9.1 (K)
- net TEMP_SENSE: now reaches IC3.24 (IO2)
- net at IC3.26 (IO4): now also R32.1
- new net: D9.2 (A), R32.2
- no-connect marks 12 -> 10

Commit message: Added new content from stream.
Other:
- note added: "2"
Changed lines of the file:
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@@
 	(generator_version "9.0")
 	(paper "A4")
+	(text "2"
+		(exclude_from_sim no)
+		(at 268.986 193.294 0)
+		(effects
+			(font
+				(size 1.27 1.27)
+			)
+		)
+	)
 	(text "ESP32"
 		(exclude_from_sim yes)

Commit message: Added new items from streams.
Parts:
- added C30: CC0603104050AAAX7R, COMPONENTS:CAP-0603, symbol COMPONENTS:CC0603104050AAAX7R
- added TP8, TP9: TP5010, CONNECTORS:5010, symbol CONNECTORS:TP5010
Connections:
- net ESP_RX: now also TP8.1
- net ESP_TX: now also TP9.1
- net GND: now also C30.2
- net TEMP_SENSE: now also C30.1
Other:
- moved on the sheet: D9, R32

Commit message: Adding new items from recent streams.
Connections:
- net INPUT_1: now also IC3.24 (IO2); no longer IC3.8 (IO32)
- net TEMP_SENSE: now also IC3.8 (IO32); no longer IC3.24 (IO2)
Other:
- moved on the sheet: C30, D8, D9, J4, R32
