File: _Projects/P0304202601-ESP32_Multi_Fan_Tester/Hardware/P0304202601-ESP32_Multi_Fan_Tester/P0304202601-ESP32.kicad_sch (KiCad schematic)
At the start: 10 parts, among them CN2 KHS4B-PH-SM4-TB(LF)(SN), IC2 ESP32-WROOM-32UE-N16

Commit message: Added new content from recent stream.
Parts:
- removed R2, R3: RC0603682075AAA, COMPONENTS:RES-0603, symbol COMPONENTS:RC0603682075AAA
- added C16: CC0603226010AABX5R, COMPONENTS:CAP-0603, symbol COMPONENTS:CC0603226010AABX5R
- added D2: TVSCDSOT23-SM712, COMPONENTS:SOT-23-3, symbol COMPONENTS:TVSCDSOT23-SM712
- added J4: KH68001-406HLF, CONNECTORS:6x1HDR2.54mm, symbol CONNECTORS:KH68001-406HLF
- added R3: RC060310K2075AAA, COMPONENTS:RES-0603, symbol COMPONENTS:RC060310K2075AAA
Connections:
- net +3.3V: now reaches R1.1
- net +3.3V: now also C2.1, C3.1, C4.1, C5.1, CN2.1, IC2.2 (3V3), C16.1, R3.1
- net ESP_EN: now reaches R1.2
- net ESP_EN: now also C1.1, IC2.3 (EN)
- net GND: now reaches C5.2
- net GND: now also C1.2, C2.2, C3.2, C4.2, CN2.4, IC2.1 (GND_1), IC2.15 (GND_2), IC2.38 (GND_3), IC2.39 (GND_4), IC2.40 (GND_5), IC2.41 (GND_6), IC2.42 (GND_7), IC2.43 (GND_8), IC2.44 (GND_9), IC2.45 (GND_10), IC2.46 (GND_11), IC2.47 (GND_12), C16.2, D2.3, J4.1
- net I2C_CLK: now reaches CN2.2
- net I2C_CLK: now also IC2.26 (IO4)
- net I2C_SDA: now reaches CN2.3
- net I2C_SDA: now also IC2.27 (IO16)
- net BOOT_MODE: now reaches IC2.25 (IO0)
- net BOOT_MODE: now also R3.2
- net ESP_RX: now reaches IC2.34 (RXD0)
- net ESP_RX: now also D2.2, J4.4
- net ESP_TX: now reaches IC2.35 (TXD0)
- net ESP_TX: now also D2.1, J4.5
- no-connect marks 0 -> 10
Other:
- moved on the sheet: C1, C2, C3, C4, C5, CN2, IC2, R1

Commit message: Added updated content that I keep forgetting to do.
Parts:
- added BOOT1, ENABLE1: SW435151014845, COMPONENTS:435151014845, symbol COMPONENTS:SW435151014845
- added D6, D7, D8: TVSCDSOT23-SM712, COMPONENTS:SOT-23-3, symbol COMPONENTS:TVSCDSOT23-SM712
- added DECREMENT1, INCREMENT1, ON/OFF1, RESET1: ~, COMPONENTS:TS14121260BK260SCRD, symbol COMPONENTS:SWTS14-1212-60-BK-260-SCR-D
- added R10, R7, R8, R9: RC060310K2075AAA, COMPONENTS:RES-0603, symbol COMPONENTS:RC060310K2075AAA
- added TP1, TP2: TP5010, CONNECTORS:5010, symbol CONNECTORS:TP5010
Connections:
- net +3.3V: now also DECREMENT1.1 (NO_1), DECREMENT1.2 (NO_2), INCREMENT1.1 (NO_1), INCREMENT1.2 (NO_2), ON/OFF1.1 (NO_1), ON/OFF1.2 (NO_2), RESET1.1 (NO_1), RESET1.2 (NO_2), TP1.1
- net BOOT_MODE: now also BOOT1.3 (COM_1), BOOT1.4 (COM_2), D6.2
- net ESP_EN: now also D6.1, ENABLE1.3 (COM_1), ENABLE1.4 (COM_2)
- net GND: now also BOOT1.1 (NO_1), BOOT1.2 (NO_2), BOOT1.5 (GND_1), BOOT1.6 (GND_2), D6.3, D7.3, D8.3, ENABLE1.1 (NO_1), ENABLE1.2 (NO_2), ENABLE1.5 (GND_1), ENABLE1.6 (GND_2), R10.2, R7.2, R8.2, R9.2, TP2.1
- net DECREMENT_SW: now reaches IC2.24 (IO2)
- net DECREMENT_SW: now also D8.1, DECREMENT1.3 (COM_1), DECREMENT1.4 (COM_2), R9.1
- net FAN_PWR_CNTROL: now reaches IC2.28 (IO17)
- net FAN_TACH: now reaches IC2.36 (IO22)
- net FAN_PWM: now reaches IC2.37 (IO23)
- net RESET_SW: now reaches IC2.4 (SENSOR_VP/IO36)
- net RESET_SW: now also D7.1, R7.1, RESET1.3 (COM_1), RESET1.4 (COM_2)
- net INCREMENT_SW: now reaches IC2.5 (SENSOR_VN/IO39)
- net INCREMENT_SW: now also D7.2, INCREMENT1.3 (COM_1), INCREMENT1.4 (COM_2), R8.1
- net TEST_CONTROL: now reaches IC2.7 (IO35)
- net TEST_CONTROL: now also D8.2, ON/OFF1.3 (COM_1), ON/OFF1.4 (COM_2), R10.1
- no-connect marks 10 -> 24
Other:
- moved on the sheet: D2, J4

Commit message: Updated files from video stream.
Parts:
- DECREMENT1, INCREMENT1, ON/OFF1: value ~ -> (none)
- MODE1: renamed from RESET1; value ~ -> (none)
Connections:
- net 5V0_FAN: now reaches IC2.30 (IO18)
- net 12V0_FAN: now reaches IC2.31 (IO19)
- net FAN_PWR_CNTROL renamed 3V3_FAN
- net RESET_SW renamed MODE_SW
- no-connect marks 24 -> 22
